File: gen3/PCBs/Micro_Breakout/Micro_Breakout.kicad_sch (KiCad schematic)
At the start: 49 parts, among them J1 BlueRobotics Depth Sensor, J10 Kill Switch, J11 StarOddi CTD Comms, J12 LED1, J13 LED2, J14 Leak Sensor, J15 Extra I2C #3, J16 Extra I2C #6, J17 Extra I2C #5, J18 Extra I2C #4, J19 GND Line, J2 Interconnect, J20 3.3V Line, J21 5V Line, J22 Extra SPI #1, J23 Extra SPI #2, J24 Extra SPI #3, J25 Secondary UART, J3 External Battery, J4 Conn_01x24, J5 External I2C, J6 Conn_01x24, J7 Extra I2C #1, J8 Extra I2C #2, J9 Lumen PWM, Q7 L78M05ABDT-TR, U1 SHT31-DIS-B, U3 MS560702BA03-50, U4 AMS1117-3_3V_C5120796, U5 MCP9808-E/MS, U6 Teensy4.1

Commit message: deleted and renamed unnecessary step and footprints
Parts:
- Q7: footprint robosub_footprints:TO-252-2_L6.5-W6.1-P4.58-LS10.0-TL -> robosub_footprints:C58069
- U1: footprint robosub_footprints:DFN-8_L2.5-W2.5-P0.50-BL-EP -> robosub_footprints:C80862
- U3: footprint robosub_footprints:SENSOR-SMD_MS560702BA03-50 -> robosub_footprints:C97627
- U4: footprint robosub_footprints:SOT-89-3_L4.5-W2.5-P1.50-LS4.2-BR -> robosub_footprints:C5120796
- U5: footprint robosub_footprints:MSOP-8_L3.0-W3.0-P0.65-LS4.9-BL -> robosub_footprints:C94847
Changed lines of the file:
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@@
 			)
 		)
-		(property "Footprint" "robosub_footprints:SOT-89-3_L4.5-W2.5-P1.50-LS4.2-BR"
+		(property "Footprint" "robosub_footprints:C5120796"
 			(at 351.79 140.97 0)
 			(effects
@@
 			)
 		)
-		(property "Footprint" "robosub_footprints:MSOP-8_L3.0-W3.0-P0.65-LS4.9-BL"
+		(property "Footprint" "robosub_footprints:C94847"
 			(at 201.93 55.88 0)
 			(effects
@@
 			)
 		)
-		(property "Description" "MCP9808-E{slash}MS (LCSC C94847)"
+		(property "Description" "MCP9808-E/MS (LCSC C94847)"
 			(at 201.93 45.72 0)
 			(effects
@@
 			)
 		)
-		(property "Footprint" "robosub_footprints:TO-252-2_L6.5-W6.1-P4.58-LS10.0-TL"
+		(property "Footprint" "robosub_footprints:C58069"
 			(at 353.06 113.03 0)
 			(effects
@@
 			)
 		)
-		(property "Footprint" "robosub_footprints:SENSOR-SMD_MS560702BA03-50"
+		(property "Footprint" "robosub_footprints:C97627"
 			(at 354.33 57.15 0)
 			(effects
@@
 			)
 		)
-		(property "Footprint" "robosub_footprints:DFN-8_L2.5-W2.5-P0.50-BL-EP"
+		(property "Footprint" "robosub_footprints:C80862"
 			(at 275.59 58.42 0)
 			(effects

Commit message: fixed
Parts:
- J1, J11, J15, J16, J17, J18, J25, J7, J8: footprint robosub_footprints:CONN_SD-43045-005_04_MOL -> robosub_footprints:430450412
- J10, J12, J13, J9: footprint robosub_footprints:CONN_SD-43045-005_02_MOL -> robosub_footprints:430450212
- J2: footprint robosub_footprints:SULLINS_SBH11-PBPC-D05-ST-BK -> robosub_footprints:SBH11-PBPC-D05-ST-BK
- J22, J23, J24: footprint robosub_footprints:CONN_SD-43045-005_06_MOL -> robosub_footprints:430450612
- Q7: footprint robosub_footprints:C58069 -> robosub_footprints:L78M05ABDT-TR
- U1: footprint robosub_footprints:C80862 -> robosub_footprints:SHT31-DIS-B
- U3: footprint robosub_footprints:C97627 -> robosub_footprints:MS560702BA03-50
- U4: footprint robosub_footprints:C5120796 -> robosub_footprints:AMS1117-3_3V_C5120796
- U5: value MCP9808-E/MS -> MCP9808-E_MS; footprint robosub_footprints:C94847 -> robosub_footprints:MCP9808-E_MS; symbol robosub_symbols:MCP9808-E/MS -> robosub_symbols:MCP9808-E_MS
- U6: value Teensy4.1 -> Teensy4_1; footprint robosub_footprints:Teensy41 -> robosub_footprints:Teensy4_1; symbol robosub_symbols:Teensy4.1 -> robosub_symbols:Teensy4_1
Changed lines of the file:
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@@
 	)
 	(symbol
-		(lib_id "robosub_symbols:Teensy4.1")
+		(lib_id "robosub_symbols:Teensy4_1")
 		(at 69.85 76.2 0)
 		(unit 1)
@@
 			)
 		)
-		(property "Value" "Teensy4.1"
+		(property "Value" "Teensy4_1"
 			(at 69.85 19.812 0)
 			(effects
@@
 			)
 		)
-		(property "Footprint" "robosub_footprints:Teensy41"
+		(property "Footprint" "robosub_footprints:Teensy4_1"
 			(at 59.69 66.04 0)
 			(effects
@@
 			)
 		)
-		(property "Description" "Symbol for Teensy4.1"
+		(property "Description" "Symbol for Teensy4_1"
 			(at 69.85 76.2 0)
 			(effects
@@
 			)
 		)
-		(property "Footprint" "robosub_footprints:C5120796"
+		(property "Footprint" "robosub_footprints:AMS1117-3_3V_C5120796"
 			(at 351.79 140.97 0)
 			(effects
@@
 			)
 		)
-		(property "Footprint" "robosub_footprints:CONN_SD-43045-005_06_MOL"
+		(property "Footprint" "robosub_footprints:430450612"
 			(at 191.77 172.72 0)
 			(effects
@@
 			)
 		)
-		(property "Footprint" "robosub_footprints:CONN_SD-43045-005_02_MOL"
+		(property "Footprint" "robosub_footprints:430450212"
 			(at 221.742 115.57 0)
 			(effects
@@
 			)
 		)
-		(property "Footprint" "robosub_footprints:CONN_SD-43045-005_02_MOL"
+		(property "Footprint" "robosub_footprints:430450212"
 			(at 189.738 115.062 0)
 			(effects
@@
 			)
 		)
-		(property "Footprint" "robosub_footprints:CONN_SD-43045-005_02_MOL"
+		(property "Footprint" "robosub_footprints:430450212"
 			(at 251.968 115.57 0)
 			(effects
@@
 			)
 		)
-		(property "Footprint" "robosub_footprints:CONN_SD-43045-005_06_MOL"
+		(property "Footprint" "robosub_footprints:430450612"
 			(at 227.33 172.72 0)
 			(effects
@@
 			)
 		)
-		(property "Footprint" "robosub_footprints:CONN_SD-43045-005_02_MOL"
+		(property "Footprint" "robosub_footprints:430450212"
 			(at 255.016 127 0)
 			(effects
@@
 			)
 		)
-		(property "Footprint" "robosub_footprints:CONN_SD-43045-005_04_MOL"
+		(property "Footprint" "robosub_footprints:430450412"
 			(at 275.59 220.98 0)
 			(effects
@@
 	)
 	(symbol
-		(lib_id "robosub_symbols:MCP9808-E/MS")
+		(lib_id "robosub_symbols:MCP9808-E_MS")
 		(at 201.93 45.72 0)
 		(unit 1)
@@
 			)
 		)
-		(property "Value" "MCP9808-E/MS"
+		(property "Value" "MCP9808-E_MS"
 			(at 201.93 38.1 0)
 			(effects
@@
 			)
 		)
-		(property "Footprint" "robosub_footprints:C94847"
+		(property "Footprint" "robosub_footprints:MCP9808-E_MS"
 			(at 201.93 55.88 0)
 			(effects
@@
 			)
 		)
-		(property "Description" "MCP9808-E/MS (LCSC C94847)"
+		(property "Description" "MCP9808-E_MS (LCSC C94847)"
 			(at 201.93 45.72 0)
 			(effects
@@
 			)
 		)
-		(property "Footprint" "robosub_footprints:CONN_SD-43045-005_04_MOL"
+		(property "Footprint" "robosub_footprints:430450412"
 			(at 275.59 201.93 0)
 			(effects
@@
 			)
 		)
-		(property "Footprint" "robosub_footprints:CONN_SD-43045-005_04_MOL"
+		(property "Footprint" "robosub_footprints:430450412"
 			(at 306.07 182.88 0)
 			(effects
@@
 			)
 		)
-		(property "Footprint" "robosub_footprints:C58069"
+		(property "Footprint" "robosub_footprints:L78M05ABDT-TR"
 			(at 353.06 113.03 0)
 			(effects
@@
 			)
 		)
-		(property "Footprint" "robosub_footprints:CONN_SD-43045-005_06_MOL"
+		(property "Footprint" "robosub_footprints:430450612"
 			(at 191.77 205.74 0)
 			(effects
@@
 			)
 		)
-		(property "Footprint" "robosub_footprints:CONN_SD-43045-005_04_MOL"
+		(property "Footprint" "robosub_footprints:430450412"
 			(at 239.776 92.71 0)
 			(effects
@@
 			)
 		)
-		(property "Footprint" "robosub_footprints:CONN_SD-43045-005_04_MOL"
+		(property "Footprint" "robosub_footprints:430450412"
 			(at 275.59 182.88 0)
 			(effects
@@
 			)
 		)
-		(property "Footprint" "robosub_footprints:CONN_SD-43045-005_04_MOL"
+		(property "Footprint" "robosub_footprints:430450412"
 			(at 360.68 207.01 0)
 			(effects
@@
 			)
 		)
-		(property "Footprint" "robosub_footprints:C97627"
+		(property "Footprint" "robosub_footprints:MS560702BA03-50"
 			(at 354.33 57.15 0)
 			(effects
@@
 			)
 		)
-		(property "Footprint" "robosub_footprints:C80862"
+		(property "Footprint" "robosub_footprints:SHT31-DIS-B"
 			(at 275.59 58.42 0)
 			(effects
@@
 			)
 		)
-		(property "Footprint" "robosub_footprints:CONN_SD-43045-005_04_MOL"
+		(property "Footprint" "robosub_footprints:430450412"
 			(at 306.07 201.93 0)
 			(effects
@@
 			)
 		)
-		(property "Footprint" "robosub_footprints:CONN_SD-43045-005_04_MOL"
+		(property "Footprint" "robosub_footprints:430450412"
 			(at 306.07 220.98 0)
 			(effects
@@
 			)
 		)
-		(property "Footprint" "robosub_footprints:CONN_SD-43045-005_04_MOL"
+		(property "Footprint" "robosub_footprints:430450412"
 			(at 187.96 92.456 0)
 			(effects
@@
 			)
 		)
-		(property "Footprint" "robosub_footprints:SULLINS_SBH11-PBPC-D05-ST-BK"
+		(property "Footprint" "robosub_footprints:SBH11-PBPC-D05-ST-BK"
 			(at 358.14 184.15 0)
 			(effects

Commit message: wired correctly gen3 sub
Connections:
- net +3.3V: now also U1.5 (VDD), U3.1 (VDD), U3.2 (PS), U3.4 (CSB), U3.5 (CSB)
- net GND: now also U1.2 (ADDR), U1.7 (R), U1.8 (VSS), U1.9 (EPAD), U3.3 (GND)
- net I2C1_SCL: now also U1.4 (SCL), U3.8 (SCLK)
- net I2C1_SDA: now also U1.1 (SDA), U3.7 (SDI/SDA)
- no-connect marks 25 -> 28
Other:
- note added: "I2C @ 0x44 default is 0x44 when ADDR is LOW"
- note added: "I2C @ 0x77 default is 0x77 when CSB is HIGH"
- moved on the sheet: J1, J10, J11, J12, J13, J14, J9, R10, R11, U1, U3, U5

Commit message: fixed cap on microbreakout
Parts:
- added C6, C7, C8: 0.1uF, Capacitor_SMD:C_0805_2012Metric_Pad1.18x1.45mm_HandSolder, symbol Device:C
Connections:
- net +3.3V: now also C6.1, C7.1, C8.1
- net GND: now also C6.2, C7.2, C8.2
Other:
- moved on the sheet: U5
