File: gen3/PCBs/Micro_Breakout/Micro_Breakout.kicad_pcb (KiCad board)
At the start: 2 copper layers, 123.5 x 83 mm, 49 parts, among them J1 BlueRobotics Depth Sensor, J10 Kill Switch, J11 StarOddi CTD Comms, J12 LED1, J13 LED2, J14 Leak Sensor, J15 Extra I2C #3, J16 Extra I2C #6, J17 Extra I2C #5, J18 Extra I2C #4, J19 GND Line, J2 Interconnect, J20 3.3V Line, J21 5V Line, J22 Extra SPI #1, J23 Extra SPI #2, J24 Extra SPI #3, J25 Secondary UART, J3 External Battery, J4 Conn_01x24, J5 External I2C, J6 Conn_01x24, J7 Extra I2C #1, J8 Extra I2C #2, J9 Lumen PWM, Q7 L78M05ABDT-TR, U1 SHT31-DIS-B, U3 MS560702BA03-50, U4 AMS1117-3_3V_C5120796, U5 MCP9808-E/MS, U6 Teensy4.1

Commit message: deleted and renamed unnecessary step and footprints
Parts:
- Q7: footprint robosub_footprints:TO-252-2_L6.5-W6.1-P4.58-LS10.0-TL -> robosub_footprints:C58069
- U1: footprint robosub_footprints:DFN-8_L2.5-W2.5-P0.50-BL-EP -> robosub_footprints:C80862
- U3: footprint robosub_footprints:SENSOR-SMD_MS560702BA03-50 -> robosub_footprints:C97627
- U4: footprint robosub_footprints:SOT-89-3_L4.5-W2.5-P1.50-LS4.2-BR -> robosub_footprints:C5120796
- U5: footprint robosub_footprints:MSOP-8_L3.0-W3.0-P0.65-LS4.9-BL -> robosub_footprints:C94847
Changed lines of the file:
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@@
 		)
 	)
-	(footprint "robosub_footprints:TO-252-2_L6.5-W6.1-P4.58-LS10.0-TL"
+	(footprint "robosub_footprints:C58069"
 		(layer "F.Cu")
 		(at 76 74 90)
@@
 			)
 		)
-		(property "Datasheet" "https://item.szlcsc.com/82618.html"
+		(property "Datasheet" "https://jlcpcb.com/partdetail/STMicroelectronics-L78M05ABDTTR/C58069"
 			(at 0 0 90)
 			(layer "F.Fab")
@@
 		)
 	)
-	(footprint "robosub_footprints:SENSOR-SMD_MS560702BA03-50"
+	(footprint "robosub_footprints:C97627"
 		(layer "F.Cu")
 		(at 42.900051 79.124968)
@@
 			)
 		)
-		(property "Datasheet" "https://item.szlcsc.com/98835.html"
+		(property "Datasheet" "https://jlcpcb.com/partdetail/TEConnectivity-MS560702BA0350/C97627"
 			(at 0 0 0)
 			(layer "F.Fab")
@@
 		)
 	)
-	(footprint "robosub_footprints:DFN-8_L2.5-W2.5-P0.50-BL-EP"
+	(footprint "robosub_footprints:C80862"
 		(layer "F.Cu")
 		(at 52.340274 78.137968)
@@
 			)
 		)
-		(property "Datasheet" "https://list.szlcsc.com/catalog/922.html"
+		(property "Datasheet" "https://jlcpcb.com/partdetail/Sensirion-SHT31_DIS_B25kS/C80862"
 			(at 0 0 0)
 			(layer "F.Fab")
@@
 		)
 	)
-	(footprint "robosub_footprints:SOT-89-3_L4.5-W2.5-P1.50-LS4.2-BR"
+	(footprint "robosub_footprints:C5120796"
 		(layer "F.Cu")
 		(at 42.985993 73.097918)
@@
 			)
 		)
-		(property "Datasheet" "https://item.szlcsc.com/421845.html"
+		(property "Datasheet" "https://jlcpcb.com/partdetail/MSKSEMI-AMS1117_33V/C5120796"
 			(at 0 0 0)
 			(layer "F.Fab")
@@
 		)
 	)
-	(footprint "robosub_footprints:MSOP-8_L3.0-W3.0-P0.65-LS4.9-BL"
+	(footprint "robosub_footprints:C94847"
 		(layer "F.Cu")
 		(at 53.131117 72.596419)

Commit message: fixed
Parts:
- J1, J11, J15, J16, J17, J18, J25, J7, J8: footprint robosub_footprints:CONN_SD-43045-005_04_MOL -> robosub_footprints:430450412
- J10, J12, J13, J9: footprint robosub_footprints:CONN_SD-43045-005_02_MOL -> robosub_footprints:430450212
- J2: footprint robosub_footprints:SULLINS_SBH11-PBPC-D05-ST-BK -> robosub_footprints:SBH11-PBPC-D05-ST-BK
- J22, J23, J24: footprint robosub_footprints:CONN_SD-43045-005_06_MOL -> robosub_footprints:430450612
- Q7: footprint robosub_footprints:C58069 -> robosub_footprints:L78M05ABDT-TR
- U1: footprint robosub_footprints:C80862 -> robosub_footprints:SHT31-DIS-B
- U3: footprint robosub_footprints:C97627 -> robosub_footprints:MS560702BA03-50
- U4: footprint robosub_footprints:C5120796 -> robosub_footprints:AMS1117-3_3V_C5120796
- U5: footprint robosub_footprints:C94847 -> robosub_footprints:MCP9808-E_MS
- U6: footprint robosub_footprints:Teensy41 -> robosub_footprints:Teensy4_1
Changed lines of the file:
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@@
 	(net 87 "unconnected-(U3-SDI{slash}SDA-Pad7)")
 	(net 88 "unconnected-(U3-VDD-Pad1)")
-	(footprint "robosub_footprints:CONN_SD-43045-005_04_MOL"
+	(footprint "robosub_footprints:430450412"
 		(layer "F.Cu")
 		(at 98 88.5 90)
@@
 		)
 	)
-	(footprint "robosub_footprints:CONN_SD-43045-005_06_MOL"
+	(footprint "robosub_footprints:430450612"
 		(layer "F.Cu")
 		(at 119.500399 91.581498)
@@
 		)
 	)
-	(footprint "robosub_footprints:CONN_SD-43045-005_04_MOL"
+	(footprint "robosub_footprints:430450412"
 		(layer "F.Cu")
 		(at 134.839999 91.499999)
@@
 		)
 	)
-	(footprint "robosub_footprints:CONN_SD-43045-005_04_MOL"
+	(footprint "robosub_footprints:430450412"
 		(layer "F.Cu")
 		(at 98 66.5 90)
@@
 		(embedded_fonts no)
 	)
-	(footprint "robosub_footprints:CONN_SD-43045-005_02_MOL"
+	(footprint "robosub_footprints:430450212"
 		(layer "F.Cu")
 		(at 160.339598 73.999999)
@@
 		)
 	)
-	(footprint "robosub_footprints:CONN_SD-43045-005_04_MOL"
+	(footprint "robosub_footprints:430450412"
 		(layer "F.Cu")
 		(at 98 110.5 90)
@@
 		)
 	)
-	(footprint "robosub_footprints:CONN_SD-43045-005_02_MOL"
+	(footprint "robosub_footprints:430450212"
 		(layer "F.Cu")
 		(at 141.3396 73.94)
@@
 		)
 	)
-	(footprint "robosub_footprints:CONN_SD-43045-005_02_MOL"
+	(footprint "robosub_footprints:430450212"
 		(layer "F.Cu")
 		(at 150.8396 73.999999)
@@
 		)
 	)
-	(footprint "robosub_footprints:CONN_SD-43045-005_04_MOL"
+	(footprint "robosub_footprints:430450412"
 		(layer "F.Cu")
 		(at 147.499999 57.059998)
@@
 		)
 	)
-	(footprint "robosub_footprints:Teensy41"
+	(footprint "robosub_footprints:Teensy4_1"
 		(layer "F.Cu")
 		(at 138.818238 114.92 180)
@@
 		)
 	)
-	(footprint "robosub_footprints:C58069"
+	(footprint "robosub_footprints:L78M05ABDT-TR"
 		(layer "F.Cu")
 		(at 76 74 90)
@@
 		)
 	)
-	(footprint "robosub_footprints:CONN_SD-43045-005_06_MOL"
+	(footprint "robosub_footprints:430450612"
 		(layer "F.Cu")
 		(at 119.499999 56.999999)
@@
 		)
 	)
-	(footprint "robosub_footprints:C97627"
+	(footprint "robosub_footprints:MS560702BA03-50"
 		(layer "F.Cu")
 		(at 42.900051 79.124968)
@@
 		)
 	)
-	(footprint "robosub_footprints:CONN_SD-43045-005_04_MOL"
+	(footprint "robosub_footprints:430450412"
 		(layer "F.Cu")
 		(at 98 99.500001 90)
@@
 		)
 	)
-	(footprint "robosub_footprints:C80862"
+	(footprint "robosub_footprints:SHT31-DIS-B"
 		(layer "F.Cu")
 		(at 52.340274 78.137968)
@@
 		)
 	)
-	(footprint "robosub_footprints:CONN_SD-43045-005_04_MOL"
+	(footprint "robosub_footprints:430450412"
 		(layer "F.Cu")
 		(at 98 77.5 90)
@@
 		)
 	)
-	(footprint "robosub_footprints:CONN_SD-43045-005_02_MOL"
+	(footprint "robosub_footprints:430450212"
 		(layer "F.Cu")
 		(at 131.839598 73.94)
@@
 		)
 	)
-	(footprint "robosub_footprints:C5120796"
+	(footprint "robosub_footprints:AMS1117-3_3V_C5120796"
 		(layer "F.Cu")
 		(at 42.985993 73.097918)
@@
 		)
 	)
-	(footprint "robosub_footprints:C94847"
+	(footprint "robosub_footprints:MCP9808-E_MS"
 		(layer "F.Cu")
 		(at 53.131117 72.596419)
@@
 		)
 	)
-	(footprint "robosub_footprints:CONN_SD-43045-005_04_MOL"
+	(footprint "robosub_footprints:430450412"
 		(layer "F.Cu")
 		(at 134.499999 57.059998)
@@
 		)
 	)
-	(footprint "robosub_footprints:CONN_SD-43045-005_04_MOL"
+	(footprint "robosub_footprints:430450412"
 		(layer "F.Cu")
 		(at 98 121.5 90)
@@
 		)
 	)
-	(footprint "robosub_footprints:CONN_SD-43045-005_06_MOL"
+	(footprint "robosub_footprints:430450612"
 		(layer "F.Cu")
 		(at 119.5 74.021499)
@@
 		)
 	)
-	(footprint "robosub_footprints:SULLINS_SBH11-PBPC-D05-ST-BK"
+	(footprint "robosub_footprints:SBH11-PBPC-D05-ST-BK"
 		(layer "B.Cu")
 		(at 153.92 89.27 180)

Commit message: Updated the whole schematic to now include 3d model
Parts:
- U5: value MCP9808-E/MS -> MCP9808-E_MS
- U6: value Teensy4.1 -> Teensy4_1
Changed lines of the file:
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@@
 		)
 		(embedded_fonts no)
-		(model "${KIPRJMOD}/3D Models/430450412.stp"
+		(model "${ROBOSUB_3D_MODELS}/430450412.stp"
 			(offset
 				(xyz -1.5 1.5 5)
@@
 			)
 		)
-		(property "Description" "430450612 (see datasheet)"
+		(property "Description" "Symbol for 430450612"
 			(at 0 0 0)
 			(layer "F.Fab")
@@
 		)
 		(embedded_fonts no)
-		(model "${KIPRJMOD}/3D Models/430450612.stp"
+		(model "${ROBOSUB_3D_MODELS}/430450612.stp"
 			(offset
 				(xyz -3 1.5 5)
@@
 		)
 		(embedded_fonts no)
-		(model "${KIPRJMOD}/3D Models/430450412.stp"
+		(model "${ROBOSUB_3D_MODELS}/430450412.stp"
 			(offset
 				(xyz -1.5 1.5 5)
@@
 		)
 		(embedded_fonts no)
-		(model "${KIPRJMOD}/3D Models/430450412.stp"
+		(model "${ROBOSUB_3D_MODELS}/430450412.stp"
 			(offset
 				(xyz -1.5 1.5 5)
@@
 		)
 		(embedded_fonts no)
-		(model "${KIPRJMOD}/3D Models/430450212.stp"
+		(model "${ROBOSUB_3D_MODELS}/430450212.stp"
 			(offset
 				(xyz 0 1.5 5)
@@
 		)
 		(embedded_fonts no)
-		(model "${KIPRJMOD}/3D Models/430450412.stp"
+		(model "${ROBOSUB_3D_MODELS}/430450412.stp"
 			(offset
 				(xyz -1.5 1.5 5)
@@
 		)
 		(embedded_fonts no)
-		(model "${KIPRJMOD}/3D Models/430450212.stp"
+		(model "${ROBOSUB_3D_MODELS}/430450212.stp"
 			(offset
 				(xyz 0 1.5 5)
@@
 		)
 		(embedded_fonts no)
-		(model "${KIPRJMOD}/3D Models/430450212.stp"
+		(model "${ROBOSUB_3D_MODELS}/430450212.stp"
 			(offset
 				(xyz 0 1.5 5)
@@
 		)
 		(embedded_fonts no)
-		(model "${KIPRJMOD}/3D Models/430450412.stp"
+		(model "${ROBOSUB_3D_MODELS}/430450412.stp"
 			(offset
 				(xyz -1.5 1.5 5)
@@
 			)
 		)
-		(property "Value" "Teensy4.1"
+		(property "Value" "Teensy4_1"
 			(at 0 10.16 0)
 			(layer "F.Fab")
@@
 			)
 		)
-		(property "Description" "Symbol for Teensy4.1"
+		(property "Description" "Symbol for Teensy4_1"
 			(at 0 0 0)
 			(layer "F.Fab")
@@
 		)
 		(embedded_fonts no)
-		(model "${KIPRJMOD}/3D Models/Teensy_4.1.step"
+		(model "${ROBOSUB_3D_MODELS}/Teensy4_1.step"
 			(offset
 				(xyz 0 0 3.762)
@@
 		)
 		(embedded_fonts no)
-		(model "C:/Users/ryota/Desktop/robosub-ee/imported_parts/robosub_3d_models/TO-252-2_L6.5-W6.1-P4.58-LS10.0-TL.step"
+		(model "${ROBOSUB_3D_MODELS}/L78M05ABDT-TR.step"
 			(offset
 				(xyz -4.030152 2.010973 0)
@@
 			)
 		)
-		(property "Description" "430450612 (see datasheet)"
+		(property "Description" "Symbol for 430450612"
 			(at 0 0 0)
 			(layer "F.Fab")
@@
 		)
 		(embedded_fonts no)
-		(model "${KIPRJMOD}/3D Models/430450612.stp"
+		(model "${ROBOSUB_3D_MODELS}/430450612.stp"
 			(offset
 				(xyz -3 1.5 5)
@@
 		)
 		(embedded_fonts no)
-		(model "packages3d/SENSOR-SMD_MS560702BA03-50.step"
+		(model "${ROBOSUB_3D_MODELS}/MS560702BA03-50.step"
 			(offset
 				(xyz 0 0 0)
@@
 		)
 		(embedded_fonts no)
-		(model "${KIPRJMOD}/3D Models/430450412.stp"
+		(model "${ROBOSUB_3D_MODELS}/430450412.stp"
 			(offset
 				(xyz -1.5 1.5 5)
@@
 		)
 		(embedded_fonts no)
-		(model "packages3d/DFN-8_L2.5-W2.5-P0.50-BL-EP.step"
+		(model "${ROBOSUB_3D_MODELS}/SHT31-DIS-B.step"
 			(offset
 				(xyz -0.0000761999988556 -0.0000761999988556 0)
@@
 		)
 		(embedded_fonts no)
-		(model "${KIPRJMOD}/3D Models/430450412.stp"
+		(model "${ROBOSUB_3D_MODELS}/430450412.stp"
 			(offset
 				(xyz -1.5 1.5 5)
@@
 		)
 		(embedded_fonts no)
-		(model "${KIPRJMOD}/3D Models/430450212.stp"
+		(model "${ROBOSUB_3D_MODELS}/430450212.stp"
 			(offset
 				(xyz 0 1.5 5)
@@
 		)
 		(embedded_fonts no)
-		(model "packages3d/SOT-89-3_L4.5-W2.5-P1.50-LS4.2-BR.step"
+		(model "${ROBOSUB_3D_MODELS}/AMS1117-3_3V_C5120796.step"
 			(offset
 				(xyz -0.2999231955 0 0)
@@
 			)
 		)
-		(property "Value" "MCP9808-E/MS"
+		(property "Value" "MCP9808-E_MS"
 			(at 0.010795 4.299975 0)
 			(layer "F.Fab")
@@
 			)
 		)
-		(property "Description" "MCP9808-E/MS (LCSC C94847)"
+		(property "Description" "MCP9808-E_MS (LCSC C94847)"
 			(at 0 0 0)
 			(layer "F.Fab")
@@
 		)
 		(embedded_fonts no)
-		(model "packages3d/MSOP-8_L3.0-W3.0-P0.65-LS4.9-BL.step"
+		(model "${ROBOSUB_3D_MODELS}/MCP9808-E_MS.step"
 			(offset
 				(xyz 0 0 0)
@@
 		)
 		(embedded_fonts no)
-		(model "${KIPRJMOD}/3D Models/430450412.stp"
+		(model "${ROBOSUB_3D_MODELS}/430450412.stp"
 			(offset
 				(xyz -1.5 1.5 5)
@@
 		)
 		(embedded_fonts no)
-		(model "${KIPRJMOD}/3D Models/430450412.stp"
+		(model "${ROBOSUB_3D_MODELS}/430450412.stp"
 			(offset
 				(xyz -1.5 1.5 5)
@@
 			)
 		)
-		(property "Description" "430450612 (see datasheet)"
+		(property "Description" "Symbol for 430450612"
 			(at 0 0 0)
 			(layer "F.Fab")
@@
 		)
 		(embedded_fonts no)
-		(model "${KIPRJMOD}/3D Models/430450612.stp"
+		(model "${ROBOSUB_3D_MODELS}/430450612.stp"
 			(offset
 				(xyz -3 1.5 5)
@@
 		)
 		(embedded_fonts no)
-		(model "${KIPRJMOD}/3D Models/SBH11-PBPC-D05-ST-BK.step"
+		(model "${ROBOSUB_3D_MODELS}/SBH11-PBPC-D05-ST-BK.step"
 			(offset
 				(xyz 0 0 0)

Commit message: wired correctly gen3 sub
Parts:
- moved C5 39.7 mm to (85.5, 63.5), turned to -90 degrees
- moved C3 37.6 mm to (85.5, 73.5), turned to -90 degrees
- moved C4 34.5 mm to (82.5, 73.5), turned to -90 degrees
- moved U3 34.1 mm to (75.0, 90.5), turned to 90 degrees
- moved U4 33.4 mm to (76.0, 77.9), turned to -90 degrees
- moved R3 31.3 mm to (104.5, 124.0), turned to 0 degrees
- moved U1 29.5 mm to (75.0, 97.0), turned to -90 degrees
- moved U5 24.7 mm to (75.0, 84.0), turned to -90 degrees
- moved C15 18.7 mm to (82.5, 63.5), turned to -90 degrees
- moved R4 10.0 mm to (85.5, 78.5)
- moved R5 10.0 mm to (82.5, 78.5)
- moved Q7 7.50 mm to (76.0, 66.5), turned to -90 degrees
- moved C2 4.99 mm to (85.5, 68.5)
- moved C1 4.99 mm to (82.5, 68.6)
Connections:
- U1 pad 1: unconnected-(U1-SDA-Pad1) -> I2C1_SDA
- U1 pad 2: unconnected-(U1-ADDR-Pad2) -> GND
- U1 pad 4: unconnected-(U1-SCL-Pad4) -> I2C1_SCL
- U1 pad 5: unconnected-(U1-VDD-Pad5) -> +3.3V
- U1 pad 7: unconnected-(U1-R-Pad7) -> GND
- U1 pad 8: unconnected-(U1-VSS-Pad8) -> GND
- U1 pad 9: unconnected-(U1-EPAD-Pad9) -> GND
- U3 pad 1: unconnected-(U3-VDD-Pad1) -> +3.3V
- U3 pad 2: unconnected-(U3-PS-Pad2) -> +3.3V
- U3 pad 3: unconnected-(U3-GND-Pad3) -> GND
- U3 pad 4: unconnected-(U3-CSB-Pad4) -> +3.3V
- U3 pad 5: unconnected-(U3-CSB-Pad5) -> +3.3V
- U3 pad 7: unconnected-(U3-SDI/SDA-Pad7) -> I2C1_SDA
- U3 pad 8: unconnected-(U3-SCLK-Pad8) -> I2C1_SCL
Routing:
- net UART_TX2: track 214.5 -> 65.3 mm, vias 0 -> 2
- net V_BATT: track 26.4 -> 10.6 mm
- net (no net): track 15.1 -> 0.00 mm, vias 3 -> 0
- net +3.3V: track 364.2 -> 349.7 mm, vias 7 -> 4
- net I2C2_SCL: track 81.7 -> 75.6 mm, vias 0 -> 1
- net I2C1_SCL: track 247.2 -> 241.5 mm, vias 0 -> 2
- net +5V: track 176.1 -> 181.4 mm, vias 2 -> 1
- net I2C1_SDA: track 272.1 -> 275.1 mm, vias 3 -> 2
- net I2C2_SDA: track 97.5 -> 95.1 mm
- net GND: track 4.41 -> 6.42 mm
- added copper zone on B.Cu, net GND
- added copper zone on F.Cu, net GND
Other:
- board text added: "MCP9808 (Temperature)"
- board text added: "MS560702BA03 (Pressure)"
- board text added: "SHT31 (Humidity)"
