File: gen3/PCBs/Micro_Breakout/Micro_Breakout.kicad_pcb (KiCad board)
At the start: 2 copper layers, 123.5 x 83 mm, 49 parts, among them J1 BlueRobotics Depth Sensor, J10 Kill Switch, J11 StarOddi CTD Comms, J12 LED1, J13 LED2, J14 Leak Sensor, J15 Extra I2C #3, J16 Extra I2C #6, J17 Extra I2C #5, J18 Extra I2C #4, J19 GND Line, J2 Interconnect, J20 3.3V Line, J21 5V Line, J22 Extra SPI #1, J23 Extra SPI #2, J24 Extra SPI #3, J25 Secondary UART, J3 External Battery, J4 Conn_01x24, J5 External I2C, J6 Conn_01x24, J7 Extra I2C #1, J8 Extra I2C #2, J9 Lumen PWM, Q7 L78M05ABDT-TR, U1 SHT31-DIS-B, U3 MS560702BA03-50, U4 AMS1117-3_3V_C5120796, U5 MCP9808-E_MS, U6 Teensy4_1

Commit message: fixed cap on microbreakout
Parts:
- added C6: 0.1uF, Capacitor_SMD:C_0805_2012Metric_Pad1.18x1.45mm_HandSolder, F.Cu at (72.5, 84.0)
- added C7: 0.1uF, Capacitor_SMD:C_0805_2012Metric_Pad1.18x1.45mm_HandSolder, F.Cu at (72.5, 97.0)
- added C8: 0.1uF, Capacitor_SMD:C_0805_2012Metric_Pad1.18x1.45mm_HandSolder, F.Cu at (72.5, 91.0)
- moved U3 1.53 mm to (76.4, 91.1), turned to 0 degrees
- moved U1 1.50 mm to (76.5, 97.0), turned to 90 degrees
- moved U5 1.50 mm to (76.5, 84.0), turned to 0 degrees
Routing:
- net +3.3V: track 349.7 -> 359.3 mm, vias 4 -> 7
- net GND: track 6.42 -> 15.6 mm
- net I2C1_SCL: track 241.5 -> 233.5 mm, vias 2 -> 3
- net I2C1_SDA: track 275.1 -> 273.4 mm, vias 2 -> 5
- net +5V: track 181.4 -> 180.5 mm, vias 1 -> 0
