File: gen3/PCBs/Power_Distribution/_autosave-Power_Distribution.kicad_pcb (KiCad board)
At the start: 2 copper layers, 70 parts, among them IC1 ACS713ELCTR-30A-T, IC2 ACS713ELCTR-30A-T, IC3 ACS713ELCTR-30A-T, IC4 ACS713ELCTR-30A-T, IC5 ACS713ELCTR-30A-T, IC6 ACS713ELCTR-30A-T, IC7 ACS713ELCTR-30A-T, IC8 ACS713ELCTR-30A-T, J1 Conn_01x02_Pin, J10 430450228, J11 430450228, J12 430450228, J13 430450228, J14 430450228, J15 430450228, J2 Conn_01x02_Pin, J3 SBH11-PBPC-D05-ST-BK, J4 1098169, J5 1098169, J6 1098169, J7 1098169, J8 430450228, J9 430450228, J98 Conn_01x08, J99 Conn_01x08, Q7 L78M05ABDT-TR, U1 MCP9808_MSOP, U3 AMS1117-3.3

Commit message: power dist board
Parts:
- added H5: MountingHole, MountingHole:MountingHole_3.2mm_M3, F.Cu at (252.5, 39.5)
- moved Cb8 112.0 mm to (215.0, 113.0), turned to 180 degrees
- moved Cf8 111.9 mm to (215.0, 123.0), turned to 180 degrees
- moved Cf16 111.6 mm to (220.0, 119.5)
- moved Cf7 101.2 mm to (200.0, 123.0), turned to 180 degrees
- moved Cf15 101.0 mm to (205.0, 119.5)
- moved Cb7 100.5 mm to (200.0, 112.5), turned to 180 degrees
- moved Q7 96.3 mm to (105.4, 92.5), turned to 180 degrees
- moved J1 93.5 mm to (100.7, 83.2), turned to 0 degrees
- moved Cf6 89.2 mm to (183.0, 123.0), turned to 180 degrees
- moved Cf14 89.1 mm to (188.0, 119.5)
- moved H2 86.1 mm to (229.1, 39.5), turned to 180 degrees
- moved H3 86.1 mm to (237.0, 39.5), turned to 180 degrees
- moved H4 86.1 mm to (244.9, 39.5), turned to 180 degrees
- moved U3 83.0 mm to (121.0, 92.0), turned to 0 degrees
- moved Cf13 79.4 mm to (173.0, 119.5)
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Routing:
- net +5V: track 0.00 -> 28.0 mm, vias 0 -> 3
- net +BATT: track 0.00 -> 20.7 mm
- net -BATT: track 0.00 -> 19.8 mm
