File: gen3/PCBs/Power_Distribution/_autosave-Power_Distribution.kicad_pcb (KiCad board)
At the start: 2 copper layers, 130 x 80 mm, 71 parts, among them IC1 ACS713ELCTR-30A-T, IC2 ACS713ELCTR-30A-T, IC3 ACS713ELCTR-30A-T, IC4 ACS713ELCTR-30A-T, IC5 ACS713ELCTR-30A-T, IC6 ACS713ELCTR-30A-T, IC7 ACS713ELCTR-30A-T, IC8 ACS713ELCTR-30A-T, J1 Conn_01x02_Pin, J10 430450228, J11 430450228, J12 430450228, J13 430450228, J14 430450228, J15 430450228, J2 Conn_01x02_Pin, J3 SBH11-PBPC-D05-ST-BK, J4 1098169, J5 1098169, J6 1098169, J7 1098169, J8 430450228, J9 430450228, J98 Conn_01x08, J99 Conn_01x08, Q7 L78M05ABDT-TR, U1 MCP9808_MSOP, U3 AMS1117-3.3

Commit message: WIP
Parts:
- moved H2 1.37 mm to (228.8, 75.9)
- moved H3 0.68 mm to (228.9, 148.4)
- turned J3 to 180 degrees
Changed lines of the file:
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@@
 	(footprint "MountingHole:MountingHole_3.2mm_M3"
 		(layer "F.Cu")
-		(at 230 76.5 180)
+		(at 228.78 75.87 180)
 		(descr "Mounting Hole 3.2mm, M3, no annular, generated by kicad-footprint-generator mountinghole.py")
 		(tags "mountinghole M3")
@@
 	(footprint "MountingHole:MountingHole_3.2mm_M3"
 		(layer "F.Cu")
-		(at 229 147.75 180)
+		(at 228.95 148.43 180)
 		(descr "Mounting Hole 3.2mm, M3, no annular, generated by kicad-footprint-generator mountinghole.py")
 		(tags "mountinghole M3")
@@
 	(footprint "Imported_Footprints:SULLINS_SBH11-PBPC-D05-ST-BK"
 		(layer "F.Cu")
-		(at 180 79.02)
+		(at 180 79.02 180)
 		(property "Reference" "J3"
 			(at 11.75 -3.77 0)
@@
 		)
 		(property "PARTREV" "J"
-			(at 0 0 0)
+			(at 0 0 180)
 			(unlocked yes)
 			(layer "F.Fab")
@@
 		)
 		(property "STANDARD" "Manufacturer Recommendations"
-			(at 0 0 0)
+			(at 0 0 180)
 			(unlocked yes)
 			(layer "F.Fab")
@@
 		)
 		(property "SNAPEDA_PN" "SBH11-PBPC-D05-ST-BK"
-			(at 0 0 0)
+			(at 0 0 180)
 			(unlocked yes)
 			(layer "F.Fab")
@@
 		)
 		(property "MAXIMUM_PACKAGE_HEIGHT" "9.1mm"
-			(at 0 0 0)
+			(at 0 0 180)
 			(unlocked yes)
 			(layer "F.Fab")
@@
 		)
 		(property "MANUFACTURER" "Sullins Connector Solutions"
-			(at 0 0 0)
+			(at 0 0 180)
 			(unlocked yes)
 			(layer "F.Fab")
@@
 		(attr through_hole)
 		(fp_line
-			(start -10.1 -4.7)
-			(end -10.1 4.4)
+			(start 10.1 4.4)
+			(end 10.1 -4.7)
 			(stroke
 				(width 0.127)
@@
 		)
 		(fp_line
-			(start -10.1 4.4)
-			(end 10.1 4.4)
+			(start 10.1 -4.7)
+			(end -10.1 -4.7)
 			(stroke
 				(width 0.127)
@@
 		)
 		(fp_line
-			(start 10.1 -4.7)
-			(end -10.1 -4.7)
+			(start -10.1 4.4)
+			(end 10.1 4.4)
 			(stroke
 				(width 0.127)
@@
 		)
 		(fp_line
-			(start 10.1 4.4)
-			(end 10.1 -4.7)
+			(start -10.1 -4.7)
+			(end -10.1 4.4)
 			(stroke
 				(width 0.127)
@@
 		)
 		(fp_line
-			(start -10.35 -4.95)
-			(end -10.35 4.65)
+			(start 10.35 4.65)
+			(end 10.35 -4.95)
 			(stroke
 				(width 0.05)
@@
 		)
 		(fp_line
-			(start -10.35 4.65)
-			(end 10.35 4.65)
+			(start 10.35 -4.95)
+			(end -10.35 -4.95)
 			(stroke
 				(width 0.05)
@@
 		)
 		(fp_line
-			(start 10.35 -4.95)
-			(end -10.35 -4.95)
+			(start -10.35 4.65)
+			(end 10.35 4.65)
 			(stroke
 				(width 0.05)
@@
 		)
 		(fp_line
-			(start 10.35 4.65)
-			(end 10.35 -4.95)
+			(start -10.35 -4.95)
+			(end -10.35 4.65)
 			(stroke
 				(width 0.05)
@@
 		)
 		(fp_line
-			(start -10.1 -4.7)
-			(end -10.1 4.4)
+			(start 10.1 4.4)
+			(end 10.1 -4.7)
 			(stroke
 				(width 0.127)
@@
 		)
 		(fp_line
-			(start -10.1 4.4)
-			(end 10.1 4.4)
+			(start 10.1 -4.7)
+			(end -10.1 -4.7)
 			(stroke
 				(width 0.127)
@@
 		)
 		(fp_line
-			(start 10.1 -4.7)
-			(end -10.1 -4.7)
+			(start -10.1 4.4)
+			(end 10.1 4.4)
 			(stroke
 				(width 0.127)
@@
 		)
 		(fp_line
-			(start 10.1 4.4)
-			(end 10.1 -4.7)
+			(start -10.1 -4.7)
+			(end -10.1 4.4)
 			(stroke
 				(width 0.127)
@@
 		)
 		(pad "1" thru_hole rect
-			(at -5.08 1.27)
+			(at -5.08 1.27 180)
 			(size 1.508 1.508)
 			(drill 1)
@@
 		)
 		(pad "2" thru_hole circle
-			(at -5.08 -1.27)
+			(at -5.08 -1.27 180)
 			(size 1.508 1.508)
 			(drill 1)
@@
 		)
 		(pad "3" thru_hole circle
-			(at -2.54 1.27)
+			(at -2.54 1.27 180)
 			(size 1.508 1.508)
 			(drill 1)
@@
 		)
 		(pad "4" thru_hole circle
-			(at -2.54 -1.27)
+			(at -2.54 -1.27 180)
 			(size 1.508 1.508)
 			(drill 1)
@@
 		)
 		(pad "5" thru_hole circle
-			(at 0 1.27)
+			(at 0 1.27 180)
 			(size 1.508 1.508)
 			(drill 1)
@@
 		)
 		(pad "6" thru_hole circle
-			(at 0 -1.27)
+			(at 0 -1.27 180)
 			(size 1.508 1.508)
 			(drill 1)
@@
 		)
 		(pad "7" thru_hole circle
-			(at 2.54 1.27)
+			(at 2.54 1.27 180)
 			(size 1.508 1.508)
 			(drill 1)
@@
 		)
 		(pad "8" thru_hole circle
-			(at 2.54 -1.27)
+			(at 2.54 -1.27 180)
 			(size 1.508 1.508)
 			(drill 1)
@@
 		)
 		(pad "9" thru_hole circle
-			(at 5.08 1.27)
+			(at 5.08 1.27 180)
 			(size 1.508 1.508)
 			(drill 1)
@@
 		)
 		(pad "10" thru_hole circle
-			(at 5.08 -1.27)
+			(at 5.08 -1.27 180)
 			(size 1.508 1.508)
 			(drill 1)

Commit message: WIP
Connections:
- J3 pad 1: PWM1 -> unconnected-(J3-Pad1)
- J3 pad 10: unconnected-(J3-Pad10) -> PWM1
- J3 pad 2: PWM2 -> GND
- J3 pad 3: PWM3 -> PWM8
- J3 pad 4: PWM4 -> PWM7
- J3 pad 5: PWM5 -> PWM6
- J3 pad 6: PWM6 -> PWM5
- J3 pad 7: PWM7 -> PWM4
- J3 pad 8: PWM8 -> PWM3
- J3 pad 9: GND -> PWM2
Changed lines of the file:
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@@
 	(net 41 "PWM7")
 	(net 42 "Net-(J99-Pin_1)")
-	(net 43 "unconnected-(J3-Pad10)")
+	(net 43 "unconnected-(J3-Pad1)")
 	(net 44 "PWM8")
 	(net 45 "+3.3V")
@@
 			(layers "*.Cu" "*.Mask")
 			(remove_unused_layers no)
-			(net 36 "PWM1")
+			(net 43 "unconnected-(J3-Pad1)")
 			(pinfunction "1")
-			(pintype "passive")
+			(pintype "passive+no_connect")
 			(solder_mask_margin 0.102)
 		)
@@
 			(layers "*.Cu" "*.Mask")
 			(remove_unused_layers no)
-			(net 38 "PWM2")
+			(net 1 "GND")
 			(pinfunction "2")
 			(pintype "passive")
@@
 			(layers "*.Cu" "*.Mask")
 			(remove_unused_layers no)
-			(net 40 "PWM3")
+			(net 44 "PWM8")
 			(pinfunction "3")
 			(pintype "passive")
@@
 			(layers "*.Cu" "*.Mask")
 			(remove_unused_layers no)
-			(net 35 "PWM4")
+			(net 41 "PWM7")
 			(pinfunction "4")
 			(pintype "passive")
@@
 			(layers "*.Cu" "*.Mask")
 			(remove_unused_layers no)
-			(net 37 "PWM5")
+			(net 39 "PWM6")
 			(pinfunction "5")
 			(pintype "passive")
@@
 			(layers "*.Cu" "*.Mask")
 			(remove_unused_layers no)
-			(net 39 "PWM6")
+			(net 37 "PWM5")
 			(pinfunction "6")
 			(pintype "passive")
@@
 			(layers "*.Cu" "*.Mask")
 			(remove_unused_layers no)
-			(net 41 "PWM7")
+			(net 35 "PWM4")
 			(pinfunction "7")
 			(pintype "passive")
@@
 			(layers "*.Cu" "*.Mask")
 			(remove_unused_layers no)
-			(net 44 "PWM8")
+			(net 40 "PWM3")
 			(pinfunction "8")
 			(pintype "passive")
@@
 			(layers "*.Cu" "*.Mask")
 			(remove_unused_layers no)
-			(net 1 "GND")
+			(net 38 "PWM2")
 			(pinfunction "9")
 			(pintype "passive")
@@
 			(layers "*.Cu" "*.Mask")
 			(remove_unused_layers no)
-			(net 43 "unconnected-(J3-Pad10)")
+			(net 36 "PWM1")
 			(pinfunction "10")
-			(pintype "passive+no_connect")
+			(pintype "passive")
 			(solder_mask_margin 0.102)
 		)
