File: gen3/PCBs/Power_Distribution/Power_Distribution.kicad_sch (KiCad schematic)
At the start: 62 parts, among them IC1 ACS713ELCTR-30A-T, IC2 ACS713ELCTR-30A-T, IC3 ACS713ELCTR-30A-T, IC4 ACS713ELCTR-30A-T, IC5 ACS713ELCTR-30A-T, IC6 ACS713ELCTR-30A-T, IC7 ACS713ELCTR-30A-T, IC8 ACS713ELCTR-30A-T, J1 1098169, J10 430450228, J11 430450228, J12 430450228, J13 430450228, J14 430450228, J15 430450228, J16 430450228, J17 430450228, J18 SBH11-PBPC-D10-ST-BK, J2 1098169, J3 Conn_01x08, J4 Conn_01x02_Pin, J5 Conn_01x02_Pin, J6 1098169, J7 1098169, J9 Conn_01x08, U1 MCP9808_MSOP, U2 MCP9808_MSOP

Commit message: power dist board
Parts:
- removed J18: SBH11-PBPC-D10-ST-BK, Imported_Footprints:SULLINS_SBH11-PBPC-D10-ST-BK, symbol Imported_Symbols:SBH11-PBPC-D10-ST-BK
- removed JP1, JP2: Jumper_2_Bridged, Jumper:SolderJumper-2_P1.3mm_Bridged2Bar_RoundedPad1.0x1.5mm, symbol Jumper:Jumper_2_Bridged
- removed JP3: Jumper_3_Bridged12, Jumper:SolderJumper-3_P1.3mm_Bridged2Bar12_RoundedPad1.0x1.5mm, symbol Jumper:Jumper_3_Bridged12
- removed U2: MCP9808_MSOP, Package_SO:MSOP-8_3x3mm_P0.65mm, symbol Sensor_Temperature:MCP9808_MSOP
- added C1, C3, C5: 1 µF, Capacitor_SMD:C_0805_2012Metric, symbol Device:C
- added C2, C4, C6: 10 µF, Capacitor_SMD:C_0805_2012Metric, symbol Device:C
- added DNP1: 0, Resistor_SMD:R_0805_2012Metric, symbol Device:R_US
- added H5: MountingHole, MountingHole:MountingHole_3.2mm_M3, symbol Mechanical:MountingHole
- added J3: SBH11-PBPC-D05-ST-BK, Imported_Footprints:SULLINS_SBH11-PBPC-D05-ST-BK, symbol Imported_Symbols:SBH11-PBPC-D05-ST-BK
- added Q7: L78M05ABDT-TR, robosub_footprints:TO-252-2_L6.5-W6.1-P4.58-LS10.0-TL, symbol L78M05ABDT-TR:L78M05ABDT-TR
- added R5, R6, R7, R8: 0R, Resistor_SMD:R_0805_2012Metric_Pad1.20x1.40mm_HandSolder, symbol Device:R_US
- added U3: AMS1117-3.3, Package_TO_SOT_SMD:SOT-223-3_TabPin2, symbol Regulator_Linear:AMS1117-3.3
- R2: value 10k -> 0R; Supplier 1 https://www.digikey.com/en/products/detail/panasonic-electr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 -> (none); Supplier 1 S/N P10KACT-ND -> (none)
- renumbered J4 to J1, J14 to J10, J16 to J11, J11 to J12, J15 to J14, J17 to J15, J5 to J2, J6 to J4, J1 to J5, J2 to J6, J10 to J8, J12 to J9, J9 to J98, J3 to J99
Connections:
- net PWM0 is gone; now on net PWM1: J8.1
- net +3.3V: now also R2.2, C5.1, C6.1, R6.1, U3.2 (VO); no longer R2.1
- net +5V: now also Cb1.1, Cb2.1, Cb3.1, Cb4.1, Cb5.1, Cb6.1, Cb7.1, Cb8.1, IC1.8 (VCC), IC2.8 (VCC), IC3.8 (VCC), IC4.8 (VCC), IC5.8 (VCC), IC6.8 (VCC), IC7.8 (VCC), IC8.8 (VCC), C3.1, C4.1, DNP1.1, Q7.3 (OUT), U3.3 (VI)
- net +BATT: now also C1.1, C2.1, Q7.1 (IN)
- net -BATT: now also C1.2, C2.2, C3.2, C4.2, C5.2, C6.2, Q7.4 (GND), U3.1 (GND)
- net 5V: no longer Cb1.1, Cb2.1, Cb3.1, Cb4.1, Cb5.1, Cb6.1, Cb7.1, Cb8.1, IC1.8 (VCC), IC2.8 (VCC), IC3.8 (VCC), IC4.8 (VCC), IC5.8 (VCC), IC6.8 (VCC), IC7.8 (VCC), IC8.8 (VCC)
- net AD0: now also R8.1
- net AD1: now also R7.1
- net COM: now also R5.1
- net GND: now also J3.9, R5.2, R7.2, R8.2; no longer R2.2
- net PWM1: now also J3.1; no longer J9.1
- net PWM2: now also J9.1, J3.2; no longer J10.1
- net PWM3: now also J10.1, J3.3; no longer J11.1
- net PWM4: now also J11.1, J3.4; no longer J12.1
- net PWM5: now also J12.1, J3.5; no longer J13.1
- net PWM6: now also J13.1, J3.6; no longer J14.1
- net PWM7: now also J14.1, J3.7; no longer J15.1
- net REF: now also R2.1
- net VIout1Div: now also J98.1 (Pin_1); no longer J98.8 (Pin_8)
- net VIout2Div: now also J98.2 (Pin_2); no longer J98.7 (Pin_7)
- net VIout3Div: now also J98.3 (Pin_3); no longer J98.6 (Pin_6)
- net VIout4Div: now also J98.4 (Pin_4); no longer J98.5 (Pin_5)
- net VIout5Div: now also J98.5 (Pin_5); no longer J98.4 (Pin_4)
- net VIout6Div: now also J98.6 (Pin_6); no longer J98.3 (Pin_3)
- net VIout7Div: now also J98.7 (Pin_7); no longer J98.2 (Pin_2)
- net VIout8Div: now also J98.8 (Pin_8); no longer J98.1 (Pin_1)
- net at J99.1 (Pin_1): now also DNP1.2, R6.2
- new net PWM8: J15.1, J3.8
- no-connect marks 4 -> 2
Other:
- note added: "To fix as of 6/23/25: -- Neo pads -- capacitors between neo pixels edits as of 2/17/26: -- remove LEDs [DONE] -- connector for +batt, -batt, SDA, SCL [DONE] -- trim down the interconnect to MLU (just PWM) [DONE] -- include way to concatenate 8 analog current sensor readings for I2C -- fix capacitor names [DONE] -- V regulator, +batt down to 5V &or 3.3V [DONE]"
- note added: "Voltage Regulators"
- note removed: "I2C @ 0x1D format: 0011(A2)(A1)(A0)"
- note removed: "Integrated MCP9808 #2"
- note removed: "To fix as of 6/23/25: -- Neo pads -- capacitors between neo pixels edits as of 2/17/26: -- remove LEDs -- connector for +batt, -batt, SDA, SCL -- trim down the interconnect to MLU (just PWM) -- include way to concatenate 8 analog current sensor readings for I2C -- fix capacitor names -- V regulator, +batt down to 5V &or 3.3V -- need 2 temp sensors? -- ESC built in current sensor/temp sensor?"
- title: Test sheet -> Power distribution board
- moved on the sheet: H1, J10, J11, J12, J13, J14, J15, J8, J9, J99, R1, U1

Commit message: WIP
Connections:
- net GND: now also J3.2; no longer J3.9
- net PWM1: now also J3.10; no longer J3.1
- net PWM2: now also J3.9; no longer J3.2
- net PWM3: now also J3.8; no longer J3.3
- net PWM4: now also J3.7; no longer J3.4
- net PWM5: now also J3.6; no longer J3.5
- net PWM6: now also J3.5; no longer J3.6
- net PWM7: now also J3.4; no longer J3.7
- net PWM8: now also J3.3; no longer J3.8
Other:
- note added: "To fix as of 6/23/25: -- Neo pads -- capacitors between neo pixels edits as of 2/17/26: -- remove LEDs [DONE] -- connector for +batt, -batt, SDA, SCL [DONE] -- trim down the interconnect to MLU (just PWM) [DONE] -- include way to concatenate 8 analog current sensor readings for I2C -- fix capacitor names [DONE] -- V regulator, +batt down to 5V &or 3.3V [DONE] -- make power connectors face "up" --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"
- note removed: "To fix as of 6/23/25: -- Neo pads -- capacitors between neo pixels edits as of 2/17/26: -- remove LEDs [DONE] -- connector for +batt, -batt, SDA, SCL [DONE] -- trim down the interconnect to MLU (just PWM) [DONE] -- include way to concatenate 8 analog current sensor readings for I2C -- fix capacitor names [DONE] -- V regulator, +batt down to 5V &or 3.3V [DONE]"
- company: blame- steven.clark@stanford.edu -> blame- steven.clark@stanford.edu, zkhuang@stanford.edu
- moved on the sheet: H1, J3, R1, U1
