File: gen3/PCBs/Power_Distribution/Power_Distribution.kicad_sch (KiCad schematic)
At the start: 72 parts, among them IC1 ACS713ELCTR-30A-T, IC2 ACS713ELCTR-30A-T, IC3 ACS713ELCTR-30A-T, IC4 ACS713ELCTR-30A-T, IC5 ACS713ELCTR-30A-T, IC6 ACS713ELCTR-30A-T, IC7 ACS713ELCTR-30A-T, IC8 ACS713ELCTR-30A-T, J1 Conn_01x02_Pin, J10 430450228, J11 430450228, J12 430450228, J13 430450228, J14 430450228, J15 430450228, J2 Conn_01x02_Pin, J3 SBH11-PBPC-D05-ST-BK, J4 1098169, J5 1098169, J6 1098169, J7 1098169, J8 430450228, J9 430450228, J98 Conn_01x08, J99 Conn_01x08, Q7 L78M05ABDT-TR, U1 MCP9808_MSOP, U3 AMS1117-3.3

Commit message: power distribution board updates
Parts:
- removed R3: 2.2k Array, Imported_Footprints:2506_8x_Resistor_Array, symbol Imported_Symbols:EXB-2HV222JV
- removed R4: 3.3k Array, Imported_Footprints:2506_8x_Resistor_Array, symbol Imported_Symbols:EXB-2HV222JV
- added R10, R11, R12, R13, R14, R15, R16, R9: 2.2k, Resistor_SMD:R_0805_2012Metric, symbol Device:R_US
- added R17, R18, R19, R20, R21, R22, R23, R24: 3.3k, Resistor_SMD:R_0805_2012Metric, symbol Device:R_US
- added TP1: TestPoint, TestPoint:TestPoint_Keystone_5019_Miniature, symbol Connector:TestPoint
- J10, J11, J12, J13, J14, J15, J8, J9: value 430450228 -> 430450212
- J4, J5, J6, J7: footprint Imported_Footprints:CUI_TBL008V-1000-04BE -> Imported_Footprints:PHOENIX_1098169
- renumbered IC1 to IC0, IC2 to IC1, IC3 to IC2, IC4 to IC3, IC5 to IC4, IC6 to IC5, IC7 to IC6, IC8 to IC7
Connections:
- net PWM8 is gone; now on net PWM7: J15.1, J3.3
- net VIout8 is gone; now on net VIout7: Cf16.1, IC7.7 (VIOUT)
- net VIout8Div is gone; now on net VIout7Div: J98.8 (Pin_8)
- net -BATT: now also J4.1, J4.3, J5.1, J5.3, J6.1, J6.3, J7.1, J7.3; no longer J4.2, J4.4, J5.2, J5.4, J6.2, J6.4, J7.2, J7.4
- net GND: now also R17.2, R18.2, R19.2, R20.2, R21.2, R22.2, R23.2, R24.2, TP1.1
- net PWM1: now also J3.9, J9.1; no longer J3.10, J8.1
- net PWM2: now also J10.1, J3.8; no longer J3.9, J9.1
- net PWM3: now also J11.1, J3.7; no longer J10.1, J3.8
- net PWM4: now also J12.1, J3.6; no longer J11.1, J3.7
- net PWM5: now also J13.1, J3.5; no longer J12.1, J3.6
- net PWM6: now also J14.1, J3.4; no longer J13.1, J3.5
- net PWM7: no longer J14.1, J3.4
- net PWR1: now also IC1.3 (IP-_1), IC1.4 (IP-_2), J4.2; no longer IC0.3 (IP-_1), IC0.4 (IP-_2), J4.1
- net PWR2: now also IC2.3 (IP-_1), IC2.4 (IP-_2), J5.4; no longer IC1.3 (IP-_1), IC1.4 (IP-_2), J4.3
- net PWR3: now also IC3.3 (IP-_1), IC3.4 (IP-_2), J5.2; no longer IC2.3 (IP-_1), IC2.4 (IP-_2), J5.1
- net PWR4: now also IC4.3 (IP-_1), IC4.4 (IP-_2), J6.4; no longer IC3.3 (IP-_1), IC3.4 (IP-_2), J5.3
- net PWR5: now also IC5.3 (IP-_1), IC5.4 (IP-_2), J6.2; no longer IC4.3 (IP-_1), IC4.4 (IP-_2), J6.1
- net PWR6: now also IC6.3 (IP-_1), IC6.4 (IP-_2), J7.4; no longer IC5.3 (IP-_1), IC5.4 (IP-_2), J6.3
- net PWR7: now also IC7.3 (IP-_1), IC7.4 (IP-_2), J7.2; no longer IC6.3 (IP-_1), IC6.4 (IP-_2), J7.1
- net VIout1: now also Cf10.1, IC1.7 (VIOUT), R10.1; no longer Cf9.1, IC0.7 (VIOUT)
- net VIout1Div: now also J98.2 (Pin_2), R10.2, R18.1; no longer J98.1 (Pin_1)
- net VIout2: now also Cf11.1, IC2.7 (VIOUT), R11.1; no longer Cf10.1, IC1.7 (VIOUT)
- net VIout2Div: now also J98.3 (Pin_3), R11.2, R19.1; no longer J98.2 (Pin_2)
- net VIout3: now also Cf12.1, IC3.7 (VIOUT), R12.1; no longer Cf11.1, IC2.7 (VIOUT)
- net VIout3Div: now also J98.4 (Pin_4), R12.2, R20.1; no longer J98.3 (Pin_3)
- net VIout4: now also Cf13.1, IC4.7 (VIOUT), R13.1; no longer Cf12.1, IC3.7 (VIOUT)
- net VIout4Div: now also J98.5 (Pin_5), R13.2, R21.1; no longer J98.4 (Pin_4)
- net VIout5: now also Cf14.1, IC5.7 (VIOUT), R14.1; no longer Cf13.1, IC4.7 (VIOUT)
- net VIout5Div: now also J98.6 (Pin_6), R14.2, R22.1; no longer J98.5 (Pin_5)
- net VIout6: now also Cf15.1, IC6.7 (VIOUT), R15.1; no longer Cf14.1, IC5.7 (VIOUT)
- net VIout6Div: now also J98.7 (Pin_7), R15.2, R23.1; no longer J98.6 (Pin_6)
- net VIout7: now also R16.1; no longer Cf15.1, IC6.7 (VIOUT)
- net VIout7Div: now also R16.2, R24.1; no longer J98.7 (Pin_7)
- removed net PWR8: IC7.3 (IP-_1), IC7.4 (IP-_2), J7.3
- new net PWM0: J3.10, J8.1
- new net PWR0: IC0.3 (IP-_1), IC0.4 (IP-_2), J4.4
- new net VIout0: Cf9.1, IC0.7 (VIOUT), R9.1
- new net VIout0Div: J98.1 (Pin_1), R17.1, R9.2
Other:
- note added: "0x1B --> Temp Sensor 0x48 --> x8 ADC for current sensors"
- note removed: "0x1B --> Temp Left 0x1D --> Temp Right 0x48 --> x8 ADC"
- moved on the sheet: Cf10, Cf11, Cf12, Cf13, Cf14, Cf15, Cf16, Cf9, J4, J5, J6, J7
