File: gen3/PCBs/Power_Distribution/_autosave-Power_Distribution.kicad_sch (KiCad schematic)
At the start: 72 parts, among them IC1 ACS713ELCTR-30A-T, IC2 ACS713ELCTR-30A-T, IC3 ACS713ELCTR-30A-T, IC4 ACS713ELCTR-30A-T, IC5 ACS713ELCTR-30A-T, IC6 ACS713ELCTR-30A-T, IC7 ACS713ELCTR-30A-T, IC8 ACS713ELCTR-30A-T, J1 Conn_01x02_Pin, J10 430450228, J11 430450228, J12 430450228, J13 430450228, J14 430450228, J15 430450228, J2 Conn_01x02_Pin, J3 SBH11-PBPC-D05-ST-BK, J4 1098169, J5 1098169, J6 1098169, J7 1098169, J8 430450228, J9 430450228, J98 Conn_01x08, J99 Conn_01x08, Q7 L78M05ABDT-TR, U1 MCP9808_MSOP, U3 AMS1117-3.3

Commit message: power dist final?
Parts:
- J10, J11, J12, J13, J14, J15: value 430450228 -> 0430450212
- J4: value 1098169 -> CUI_TBL008V-1000-04BE; footprint Imported_Footprints:CUI_TBL008V-1000-04BE -> Connector_AMASS:AMASS_XT60PW-F_1x02_P7.20mm_Horizontal
- J5, J6, J7: value 1098169 -> CUI_TBL008V-1000-04BE
- J8, J9: value 430450228 -> 430450212
Changed lines of the file:
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@@
 		(on_board yes)
 		(dnp no)
-		(fields_autoplaced yes)
 		(property "Reference" "J6"
 			(at 92.71 28.7019 90)
@@
 			)
 		)
-		(property "Value" "1098169"
-			(at 92.71 31.2419 90)
+		(property "Value" "CUI_TBL008V-1000-04BE"
+			(at 78.486 22.098 90)
 			(effects
 				(font
@@
 		(on_board yes)
 		(dnp no)
-		(fields_autoplaced yes)
 		(property "Reference" "J5"
 			(at 66.04 28.9559 90)
@@
 			)
 		)
-		(property "Value" "1098169"
-			(at 66.04 31.4959 90)
+		(property "Value" "CUI_TBL008V-1000-04BE"
+			(at 51.816 22.352 90)
 			(effects
 				(font
@@
 			)
 		)
-		(property "Value" "430450228"
+		(property "Value" "0430450212"
 			(at 67.818 179.3239 0)
 			(effects
@@
 			)
 		)
-		(property "Value" "430450228"
+		(property "Value" "430450212"
 			(at 40.386 163.8299 0)
 			(effects
@@
 			)
 		)
-		(property "Value" "430450228"
+		(property "Value" "430450212"
 			(at 40.386 156.2099 0)
 			(effects
@@
 			)
 		)
-		(property "Value" "430450228"
+		(property "Value" "0430450212"
 			(at 67.818 164.0839 0)
 			(effects
@@
 			)
 		)
-		(property "Value" "430450228"
+		(property "Value" "0430450212"
 			(at 67.818 171.7039 0)
 			(effects
@@
 			)
 		)
-		(property "Value" "430450228"
+		(property "Value" "0430450212"
 			(at 40.386 179.0699 0)
 			(effects
@@
 			)
 		)
-		(property "Value" "430450228"
+		(property "Value" "0430450212"
 			(at 40.386 171.4499 0)
 			(effects
@@
 		(on_board yes)
 		(dnp no)
-		(fields_autoplaced yes)
 		(property "Reference" "J4"
 			(at 39.37 28.7019 90)
@@
 			)
 		)
-		(property "Value" "1098169"
-			(at 39.37 31.2419 90)
+		(property "Value" "CUI_TBL008V-1000-04BE"
+			(at 25.146 22.098 90)
 			(effects
 				(font
@@
 			)
 		)
-		(property "Footprint" "Imported_Footprints:CUI_TBL008V-1000-04BE"
+		(property "Footprint" "Connector_AMASS:AMASS_XT60PW-F_1x02_P7.20mm_Horizontal"
 			(at 32.766 29.972 0)
 			(effects
@@
 			)
 		)
-		(property "Value" "430450228"
+		(property "Value" "0430450212"
 			(at 67.818 156.4639 0)
 			(effects
@@
 			)
 		)
-		(property "Value" "1098169"
-			(at 118.364 30.9879 90)
+		(property "Value" "CUI_TBL008V-1000-04BE"
+			(at 104.14 21.844 90)
 			(effects
 				(font
