File: gen3/PCBs/Battery_Boards/Power_ManagementV3_eli/Power_ManagementV3_eli.kicad_pcb (KiCad board)
At the start: 2 copper layers, 244 x 107 mm, 147 parts, among them J1 Conn_01x02_Pin, J10 via, J11 Conn_01x02_Pin, J12 Conn_01x02_Pin, J13 Conn_01x04_Pin, J14 Conn_01x08, J15 Conn_01x08, J16 Conn_01x02_Pin, J17 FPGA MOUNT, J2 Conn_01x02_Pin, J3 Conn_01x08, J4 Conn_01x08, J5 Conn_01x02_Pin, J6 Conn_01x02_Pin, J9 Conn_01x04_Pin, Q1 MCTL160N15Y-TP, Q2 MCTL160N15Y-TP, Q3 MCTL160N15Y-TP, Q4 MCTL160N15Y-TP, Q5 MCTL160N15Y-TP, Q6 MCTL160N15Y-TP, U1 STPS5045SG-TR, U10 SN74HC132PWR, U11 SN74LVC1G373DCKR, U12 MCP6564-E/ST, U13 STPS5045SG-TR, U14 MCP9808_MSOP, U15 STPS5045SG-TR, U16 MCP9808_MSOP, U2 STPS5045SG-TR, U3 LTC1255CS8-PBF, U4 BA033CC0FP-E2, U5 ACS758LCB-100U-PFF-T, U6 SN74HC132PWR, U8 SN74HC132PWR, U9 SN74HC132PWR

Commit message: to_order has the 3 main pcbs consolidated. pcbs have been put into production
Parts:
- removed the H6 at (132.0, 139.1)
- removed the H7 at (59.0, 139.0)
- removed the H8 at (132.0, 42.0)
- removed the H9 at (59.0, 42.0)
- removed J11, J12: Conn_01x02_Pin, Connector_AMASS:AMASS_XT60IPW-M_1x03_P7.20mm_Horizontal
- removed J13: Conn_01x04_Pin, Imported_Footprints:CONN_SD-43045-008_04_MOL
- removed J14, J15: Conn_01x08, Connector_PinHeader_2.54mm:PinHeader_1x08_P2.54mm_Vertical
- removed J16: Conn_01x02_Pin, Connector_AMASS:AMASS_XT60PW-F_1x02_P7.20mm_Horizontal
- removed PM3: LMS78, Imported_Footprints:LMS78
- removed R27, R29, R32, R34, R36, R37, R39, R41: 10k, Resistor_SMD:R_0805_2012Metric_Pad1.20x1.40mm_HandSolder
- removed R28, R30, R38, R40: 20k, Resistor_SMD:R_0805_2012Metric_Pad1.20x1.40mm_HandSolder
- removed R31, R33, R35: 47k, Resistor_SMD:R_0805_2012Metric_Pad1.20x1.40mm_HandSolder
- removed U13, U15: STPS5045SG-TR, Imported_Footprints:D2PAK_STM
- removed U16: MCP9808_MSOP, Package_SO:MSOP-8_3x3mm_P0.65mm
Routing:
- net +BATT2_bak: track 94.1 -> 0.00 mm, vias 2 -> 0
- net /SDA: track 79.2 -> 0.00 mm
- net /SCL: track 75.5 -> 0.00 mm
- net +Backup: track 57.2 -> 0.00 mm, vias 1 -> 0
- net +BATT1_bak: track 55.1 -> 0.00 mm, vias 2 -> 0
- net /5V: track 32.6 -> 0.00 mm, vias 2 -> 0
- net GND_bak: track 30.8 -> 0.00 mm, vias 2 -> 0
- net Net-(J14-Pin_1): track 7.94 -> 0.00 mm
- net Net-(J14-Pin_2): track 7.72 -> 0.00 mm
- net Net-(J14-Pin_3): track 7.50 -> 0.00 mm
- net Net-(J15-Pin_3): track 5.16 -> 0.00 mm
- net Net-(J15-Pin_4): track 4.62 -> 0.00 mm
- net Net-(U16-SCL): track 3.44 -> 0.00 mm
- net Net-(U16-SDA): track 2.90 -> 0.00 mm
- removed copper zone on F.Cu, net +BATT1_bak
- removed copper zone on F.Cu, net +BATT2_bak
- removed copper zone on F.Cu, net +Backup
- removed copper zone on B.Cu, net GND_bak
- removed copper zone on F.Cu, net GND_bak
Other:
- board text removed: "BOTTOM SIDE OBSTRUCTED, LEFT RIGHT USED FOR SLIDING RAILS, POWER CONNECTORS AT THE TOP AND THE BUSSES ON THE SIDE"
- board text removed: "KILL SWITCH IS COMPETITION REQIUREMENT!!!!"
- board text removed: "MAKE ANOTHER DESIGN THAT IS JUST THE DIODES"
- board text removed: "is what I told myself... This is the brainless version that should hopefully be bullet proof"
