File: gen3/PCBs/to_order/to_order/to_order.kicad_pcb (KiCad board)
At the start: 2 copper layers, 261.2 x 259 mm, 213 parts, among them J1 BlueRobotics Depth Sensor, J1 Conn_01x02_Pin, J10 Kill Switch, J10 via, J11 Conn_01x02_Pin, J11 StarOddi CTD Comms, J12 Conn_01x02_Pin, J12 LED1, J13 Conn_01x02_Pin, J13 LED2, J14 Conn_01x08, J14 Leak Sensor, J15 Conn_01x08, J15 Extra I2C #3, J16 Conn_01x02_Pin, J16 Extra I2C #6, J17 Extra I2C #5, J17 FPGA MOUNT, J18 Conn_01x04_Socket, J18 Extra I2C #4, J19 GND Line, J2 Conn_01x02_Pin, J2 Interconnect, J20 3.3V Line, J21 5V Line, J21 Conn_01x02_Pin, J22 Conn_01x02_Pin, J22 Extra SPI #1, J23 Extra SPI #2, J24 Extra SPI #3, J25 Secondary UART, J3 Conn_01x08, J3 External Battery, J4 Conn_01x08, J4 Conn_01x24, J5 Conn_01x02_Pin, J5 External I2C, J6 Conn_01x02_Pin, J6 Conn_01x24, J7 Extra I2C #1, J8 Extra I2C #2, J9 Conn_01x04_Pin, J9 Lumen PWM, Q1 MCTL160N15Y-TP, Q2 MCTL160N15Y-TP, Q3 MCTL160N15Y-TP, Q4 MCTL160N15Y-TP, Q5 MCTL160N15Y-TP, Q6 MCTL160N15Y-TP, Q7 L78M05ABDT-TR, U1 STPS5045SG-TR, U10 SN74HC132PWR, U11 SN74LVC1G373DCKR, U12 MCP6564-E/ST, U14 MCP9808_MSOP, U15 AMS1117-3.3, U16 MCP9808_MSOP, U17 ACS758LCB-100U-PFF-T, U18 SRT60L100DC-R, U2 MCP9808_MSOP, U2 STPS5045SG-TR, U3 LTC1255CS8-PBF, U4 BA033CC0FP-E2, U4 BME280, U5 ACS758LCB-100U-PFF-T, U6 SN74HC132PWR, U6 Teensy4.1, U8 SN74HC132PWR, U9 SN74HC132PWR

Commit message: to_order has the 3 main pcbs consolidated. pcbs have been put into production
Parts:
- removed 2A2, 2B2, 2Y1, 3A2, 3B2, 3Y1, 4A1, 4B1, 4Y1, TP13, TP14, TP8, TP9: TestPoint, TestPoint:TestPoint_Pad_1.0x1.0mm
- removed the C1 at (101.0, 89.5)
- removed the C1 at (138.6, -87.7)
- removed C10, C11: 10,000uF, Capacitor_THT:CP_Radial_D16.0mm_P7.50mm
- removed the C12 at (102.5, 101.5)
- removed the C12 at (297.9, 79.1)
- removed the C13 at (101.5, 105.5)
- removed the C13 at (301.6, 88.4)
- removed the C14 at (105.0, 105.5)
- removed the C14 at (303.7, 88.2)
- removed the C15 at (291.7, 79.2)
- removed the C15 at (94.0, 97.0)
- removed the C2 at (121.9, -79.1)
- removed the C2 at (104.0, 89.5)
- removed C7: 0.1u, Capacitor_SMD:C_0805_2012Metric_Pad1.18x1.45mm_HandSolder
- removed C8: 100nF, Capacitor_SMD:C_0805_2012Metric_Pad1.18x1.45mm_HandSolder
- removed C9: 1µF, Capacitor_SMD:C_0805_2012Metric_Pad1.18x1.45mm_HandSolder
- removed CR1: SBRT15U50SP5-13, Imported_Footprints:POWERDI5_DIO
- removed D1, D2: D_Zener, Imported_Footprints:1N5242B
- removed D10, D11, D12, D13, D14, D4, D5, D6, D7, D8, D9: GreenLED, LED_SMD:LED_0603_1608Metric_Pad1.05x0.95mm_HandSolder
- removed D3: TVS, Diode_SMD:D_SMA
- removed the H6 at (82.0, 70.5)
- removed the H6 at (240.7, 140.6)
- removed the H6 at (144.6, -7.90)
- removed the H7 at (82.0, 144.5)
- removed the H7 at (71.6, -7.98)
- removed the H7 at (240.8, 72.6)
- removed the H8 at (322.8, 140.6)
- removed the H8 at (144.6, -105.0)
- removed the H8 at (196.5, 70.5)
- removed the H8 at (308.8, 131.6)
- removed the H8 at (254.8, 131.6)
- removed the H9 at (196.5, 144.5)
- removed the H9 at (322.8, 72.6)
- removed the H9 at (71.6, -105.0)
- removed the J1 at (75.7, -71.2)
- removed the J1 at (152.5, 73.1)
- removed the J10 at (159.3, 89.9)
- removed the J10 at (103.1, -24.6)
- removed the J11 at (165.5, 73.1)
- removed the J11 at (271.2, 71.4)
- removed the J12 at (168.8, 90.0)
- removed the J12 at (271.2, 82.4)
- removed the J13 at (260.8, 71.6)
- removed the J13 at (178.3, 90.0)
- removed the J14 at (173.0, 73.1)
- removed the J14 at (293.9, 109.3)
- removed the J15 at (116.0, 104.5)
- removed the J15 at (281.2, 109.3)
- removed the J16 at (116.0, 137.5)
- removed the J16 at (254.2, 83.9)
- removed the J17 at (116.0, 126.5)
- removed the J17 at (143.5, -21.1)
- removed the J18 at (116.0, 115.5)
- removed the J18 at (286.1, 88.6)
- removed the J2 at (75.7, -51.4)
- removed the J2 at (171.9, 105.3)
- removed the J21 at (100.0, 143.2)
- removed the J21 at (246.8, 106.1)
- removed the J22 at (246.7, 89.3)
- removed the J22 at (137.5, 73.0)
- removed the J3 at (101.2, 73.8)
- removed the J3 at (142.5, -54.1)
- removed the J4 at (142.5, -41.4)
- removed the J4 at (186.1, 119.6)
- removed the J5 at (112.5, 73.7)
- removed the J5 at (75.6, -39.0)
- removed the J6 at (186.0, 142.1)
- removed the J6 at (74.6, -17.5)
- removed the J7 at (116.0, 82.5)
- removed the J8 at (116.0, 93.5)
- removed the J9 at (73.5, -91.4)
- removed the J9 at (149.8, 89.9)
- removed JP1, JP3: SolderJumper_2_Bridged, Jumper:SolderJumper-2_P1.3mm_Bridged2Bar_RoundedPad1.0x1.5mm
- removed JP10, JP11, JP25, JP27: Jumper_2_Bridged, Jumper:SolderJumper-2_P1.3mm_Bridged2Bar_RoundedPad1.0x1.5mm
- removed JP12: Jumper_2_Open, Imported_Footprints:KEYSTONE_5102
- removed JP2: SolderJumper_2_Open, Jumper:SolderJumper-2_P1.3mm_Open_RoundedPad1.0x1.5mm
- removed JP21, JP23, JP26: Jumper_2_Open, Jumper:SolderJumper-2_P1.3mm_Open_RoundedPad1.0x1.5mm
- removed JP6, JP7: ~, Jumper:SolderJumper-2_P1.3mm_Bridged2Bar_RoundedPad1.0x1.5mm
- removed PM2: LMS78, Imported_Footprints:LMS78
- removed Q1, Q2, Q3, Q4, Q5, Q6: MCTL160N15Y-TP, Imported_Footprints:TOLL-8L_MCC
- removed the Q7 at (94.0, 90.0)
- removed the Q7 at (299.2, 73.2)
- removed the R1 at (101.0, 112.0)
- removed the R1 at (128.3, -62.4)
- removed the R10 at (140.3, -83.2)
- removed the R10 at (122.5, 128.0)
- removed the R11 at (125.3, -17.8)
- removed the R11 at (122.5, 125.0)
- removed R12, R17, R18, R19, R20, R22, R23, R24: 100, Resistor_SMD:R_0402_1005Metric
- removed R13: 2.2k, Resistor_SMD:R_0805_2012Metric_Pad1.20x1.40mm_HandSolder
- removed R14: 0.5 Ohm 25W, Imported_Footprints:TO508P1229X317-3N
- removed R15: 3.9k, Resistor_SMD:R_0805_2012Metric_Pad1.20x1.40mm_HandSolder
- removed R16: 10k, Resistor_SMD:R_0805_2012Metric_Pad1.20x1.40mm_HandSolder
- removed the R2 at (101.0, 115.0)
- removed the R2 at (125.5, -61.4)
- removed R25: 15k, Resistor_SMD:R_0402_1005Metric
- removed R26: 1.5k, Resistor_SMD:R_0402_1005Metric
- removed the R3 at (105.0, 114.0)
- removed the R3 at (128.3, -60.6)
- removed the R4 at (131.3, -90.1)
- removed the R4 at (104.0, 84.5)
- removed R42, R43, R44, R45, R9: 0R, Resistor_SMD:R_0805_2012Metric_Pad1.20x1.40mm_HandSolder
- removed the R5 at (101.0, 84.5)
- removed the R5 at (131.3, -93.6)
- removed the R6 at (135.0, -65.3)
- removed the R6 at (122.5, 137.0)
- removed the R7 at (134.0, -68.1)
- removed the R7 at (122.5, 134.0)
- removed the R8 at (132.9, -65.3)
- removed the R8 at (122.5, 131.0)
- removed S1: 100SP1T1B4M2QE, Imported_Footprints:SW_100SP1T1B4M2QE
- removed TH1, TH2: Thermistor_US, Resistor_SMD:R_0805_2012Metric
- removed U10, U8, U9: SN74HC132PWR, eli_custom_footprint_lib:SOP65P640X120-14N
- removed U11: SN74LVC1G373DCKR, Imported_Footprints:SN74LVC
- removed U12: MCP6564-E/ST, footprints:TSSOP14_MC_MCH
- removed U14: MCP9808_MSOP, Package_SO:MSOP-8_3x3mm_P0.65mm
- removed the U15 at (95.0, 104.0)
- removed the U15 at (302.5, 81.8)
- removed the U2 at (102.5, 94.5)
- removed the U2 at (139.7, -74.1)
- removed the U4 at (95.0, 113.5)
- removed the U4 at (142.2, -59.9)
- removed U5: ACS758LCB-100U-PFF-T, Imported_Footprints:Allegro_MicroSystems,_LLC-CB-5-PFF-0-0-MFG
- removed the U6 at (134.0, -30.4)
- removed the U6 at (156.8, 130.9)
- removed VR1, VR2: 3296W-1-103RLF, Imported_Footprints:TRIM_3296W-1-103RLF
- added C1: 10uF, Capacitor_SMD:C_0805_2012Metric_Pad1.18x1.45mm_HandSolder, F.Cu at (288.5, 128.0)
- added C1: 1 µF, Capacitor_SMD:C_0805_2012Metric, F.Cu at (128.1, 14.8)
- added C12: 10uF, Capacitor_SMD:C_0805_2012Metric_Pad1.18x1.45mm_HandSolder, F.Cu at (287.0, 116.0)
- added C12: 10uF, Capacitor_SMD:C_0805_2012Metric_Pad1.18x1.45mm_HandSolder, F.Cu at (153.9, 80.1)
- added C13: 10uF, Capacitor_SMD:C_0805_2012Metric_Pad1.18x1.45mm_HandSolder, F.Cu at (157.6, 89.4)
- added C13: 10uF, Capacitor_SMD:C_0805_2012Metric_Pad1.18x1.45mm_HandSolder, F.Cu at (288.0, 112.0)
- added C14: 1uF, Capacitor_SMD:C_0805_2012Metric_Pad1.18x1.45mm_HandSolder, F.Cu at (159.7, 89.2)
- added C14: 1uF, Capacitor_SMD:C_0805_2012Metric_Pad1.18x1.45mm_HandSolder, F.Cu at (284.5, 112.0)
- added C15: 10uF, Capacitor_SMD:C_0805_2012Metric_Pad1.18x1.45mm_HandSolder, F.Cu at (147.7, 80.2)
- added C15: 10uF, Capacitor_SMD:C_0805_2012Metric_Pad1.18x1.45mm_HandSolder, F.Cu at (295.5, 120.5)
- added C2: 1uF, Capacitor_SMD:C_0805_2012Metric_Pad1.18x1.45mm_HandSolder, F.Cu at (285.5, 128.0)
- added C2: 10 µF, Capacitor_SMD:C_0805_2012Metric, F.Cu at (128.1, 12.3)
- added Cb1: 0.1 µF, Capacitor_SMD:C_0805_2012Metric_Pad1.18x1.45mm_HandSolder, F.Cu at (114.3, 31.3)
- added Cb2: 0.1 µF, Capacitor_SMD:C_0805_2012Metric_Pad1.18x1.45mm_HandSolder, F.Cu at (129.4, 31.3)
- added Cb3: 0.1 µF, Capacitor_SMD:C_0805_2012Metric_Pad1.18x1.45mm_HandSolder, F.Cu at (146.4, 31.3)
- added Cb4: 0.1 µF, Capacitor_SMD:C_0805_2012Metric_Pad1.18x1.45mm_HandSolder, F.Cu at (193.3, 31.3)
- added Cb5: 0.1 µF, Capacitor_SMD:C_0805_2012Metric_Pad1.18x1.45mm_HandSolder, F.Cu at (161.3, 31.3)
- added Cb6: 0.1 µF, Capacitor_SMD:C_0805_2012Metric_Pad1.18x1.45mm_HandSolder, F.Cu at (178.3, 31.3)
- added Cb7: 0.1 µF, Capacitor_SMD:C_0805_2012Metric_Pad1.18x1.45mm_HandSolder, F.Cu at (210.3, 31.3)
- added Cb8: 0.1 µF, Capacitor_SMD:C_0805_2012Metric_Pad1.18x1.45mm_HandSolder, F.Cu at (225.3, 30.8)
- added Cf1: 100 nF, Capacitor_SMD:C_0805_2012Metric_Pad1.18x1.45mm_HandSolder, F.Cu at (118.6, 38.1)
- added Cf10: 1 µF, Capacitor_SMD:C_0805_2012Metric_Pad1.18x1.45mm_HandSolder, F.Cu at (133.6, 35.6)
- added Cf11: 1 µF, Capacitor_SMD:C_0805_2012Metric_Pad1.18x1.45mm_HandSolder, F.Cu at (150.6, 35.6)
- added Cf12: 1 µF, Capacitor_SMD:C_0805_2012Metric_Pad1.18x1.45mm_HandSolder, F.Cu at (165.6, 35.6)
- added Cf13: 1 µF, Capacitor_SMD:C_0805_2012Metric_Pad1.18x1.45mm_HandSolder, F.Cu at (182.6, 35.6)
- added Cf14: 1 µF, Capacitor_SMD:C_0805_2012Metric_Pad1.18x1.45mm_HandSolder, F.Cu at (197.6, 35.6)
- added Cf15: 1 µF, Capacitor_SMD:C_0805_2012Metric_Pad1.18x1.45mm_HandSolder, F.Cu at (214.6, 35.6)
- added Cf16: 1 µF, Capacitor_SMD:C_0805_2012Metric_Pad1.18x1.45mm_HandSolder, F.Cu at (229.6, 35.6)
- added Cf2: 100 nF, Capacitor_SMD:C_0805_2012Metric_Pad1.18x1.45mm_HandSolder, F.Cu at (133.6, 38.1)
- added Cf3: 100 nF, Capacitor_SMD:C_0805_2012Metric_Pad1.18x1.45mm_HandSolder, F.Cu at (150.6, 37.8)
- added Cf4: 100 nF, Capacitor_SMD:C_0805_2012Metric_Pad1.18x1.45mm_HandSolder, F.Cu at (165.6, 38.1)
- added Cf5: 100 nF, Capacitor_SMD:C_0805_2012Metric_Pad1.18x1.45mm_HandSolder, F.Cu at (182.7, 37.9)
- added Cf6: 100 nF, Capacitor_SMD:C_0805_2012Metric_Pad1.18x1.45mm_HandSolder, F.Cu at (197.7, 37.9)
- added Cf7: 100 nF, Capacitor_SMD:C_0805_2012Metric_Pad1.18x1.45mm_HandSolder, F.Cu at (214.7, 37.9)
- added Cf8: 100 nF, Capacitor_SMD:C_0805_2012Metric_Pad1.18x1.45mm_HandSolder, F.Cu at (229.7, 37.9)
- added Cf9: 1 µF, Capacitor_SMD:C_0805_2012Metric_Pad1.18x1.45mm_HandSolder, F.Cu at (118.6, 35.6)
- added DNP1: 0, Resistor_SMD:R_0805_2012Metric, F.Cu at (150.2, -3.57)
- added H2: MountingHole, MountingHole:MountingHole_4.3mm_M4, F.Cu at (239.2, -8.81)
- added H3: MountingHole, MountingHole:MountingHole_4.3mm_M4, F.Cu at (239.2, 62.0)
- added H4: MountingHole, MountingHole:MountingHole_4.3mm_M4, F.Cu at (97.0, -8.81)
- added H5: MountingHole, MountingHole:MountingHole_4.3mm_M4, F.Cu at (97.0, 62.0)
- added H6: MountingHole, MountingHole:MountingHole_4.3mm_M4, F.Cu at (307.5, 147.0)
- added H6: MountingHole, MountingHole:MountingHole_4.3mm_M4, F.Cu at (96.7, 141.6)
- added H7: MountingHole, MountingHole:MountingHole_4.3mm_M4, F.Cu at (96.8, 73.6)
- added H7: MountingHole, MountingHole:MountingHole_4.3mm_M4, F.Cu at (307.5, 73.0)
- added H8: MountingHole, MountingHole:MountingHole_4.3mm_M4, F.Cu at (178.8, 141.6)
- added H8: MountingHole, MountingHole:MountingHole_4.3mm_M4, F.Cu at (193.0, 147.0)
- added H8: MountingHole, MountingHole:MountingHole_4.3mm_M4, B.Cu at (110.8, 132.6)
- added H8: MountingHole, MountingHole:MountingHole_4.3mm_M4, B.Cu at (164.8, 132.6)
- added H9: MountingHole, MountingHole:MountingHole_4.3mm_M4, F.Cu at (178.8, 73.6)
- added H9: MountingHole, MountingHole:MountingHole_4.3mm_M4, F.Cu at (193.0, 73.0)
- added IC1: ACS713ELCTR-30A-T, Imported_Footprints:ACS711ELCTR25ABT, F.Cu at (111.6, 36.3)
- added IC2: ACS713ELCTR-30A-T, Imported_Footprints:ACS711ELCTR25ABT, F.Cu at (126.6, 36.3)
- added IC3: ACS713ELCTR-30A-T, Imported_Footprints:ACS711ELCTR25ABT, F.Cu at (143.6, 36.3)
- added IC4: ACS713ELCTR-30A-T, Imported_Footprints:ACS711ELCTR25ABT, F.Cu at (158.6, 36.3)
- added IC5: ACS713ELCTR-30A-T, Imported_Footprints:ACS711ELCTR25ABT, F.Cu at (175.6, 36.3)
- added IC6: ACS713ELCTR-30A-T, Imported_Footprints:ACS711ELCTR25ABT, F.Cu at (190.6, 36.3)
- added IC7: ACS713ELCTR-30A-T, Imported_Footprints:ACS711ELCTR25ABT, F.Cu at (207.6, 36.3)
- added IC8: ACS713ELCTR-30A-T, Imported_Footprints:ACS711ELCTR25ABT, F.Cu at (222.6, 36.3)
- added J1: Conn_01x02_Pin, Connector_AMASS:AMASS_XT60IPW-M_1x03_P7.20mm_Horizontal, F.Cu at (111.7, -2.35)
- added J1: BlueRobotics Depth Sensor, Imported_Footprints:CONN_SD-43045-005_04_MOL, F.Cu at (237.0, 144.4)
- added J10: 430450228, Connector_Molex:Molex_Micro-Fit_3.0_43045-0212_2x01_P3.00mm_Vertical, F.Cu at (175.8, 14.8)
- added J10: Kill Switch, Imported_Footprints:CONN_SD-43045-005_02_MOL, F.Cu at (230.2, 127.6)
- added J11: StarOddi CTD Comms, Imported_Footprints:CONN_SD-43045-005_04_MOL, F.Cu at (224.0, 144.4)
- added J11: 430450228, Connector_Molex:Molex_Micro-Fit_3.0_43045-0212_2x01_P3.00mm_Vertical, F.Cu at (185.8, 14.8)
- added J11: Conn_01x02_Pin, Connector_AMASS:AMASS_XT60IPW-M_1x03_P7.20mm_Horizontal, B.Cu at (127.2, 72.4)
- added J12: LED1, Imported_Footprints:CONN_SD-43045-005_02_MOL, F.Cu at (220.7, 127.5)
- added J12: 430450228, Connector_Molex:Molex_Micro-Fit_3.0_43045-0212_2x01_P3.00mm_Vertical, F.Cu at (195.8, 14.8)
- added J12: Conn_01x02_Pin, Connector_AMASS:AMASS_XT60IPW-M_1x03_P7.20mm_Horizontal, B.Cu at (127.2, 83.4)
- added J13: LED2, Imported_Footprints:CONN_SD-43045-005_02_MOL, F.Cu at (211.2, 127.5)
- added J13: Conn_01x02_Pin, Connector_AMASS:AMASS_XT30PW-F_1x02_P2.50mm_Horizontal, F.Cu at (116.8, 72.6)
- added J13: 430450228, Connector_Molex:Molex_Micro-Fit_3.0_43045-0212_2x01_P3.00mm_Vertical, F.Cu at (205.8, 14.8)
- added J14: Leak Sensor, Connector_PinHeader_2.54mm:PinHeader_1x03_P2.54mm_Vertical, F.Cu at (216.5, 144.4)
- added J14: 430450228, Connector_Molex:Molex_Micro-Fit_3.0_43045-0212_2x01_P3.00mm_Vertical, F.Cu at (215.8, 14.8)
- added J14: Conn_01x08, Connector_PinHeader_2.54mm:PinHeader_1x08_P2.54mm_Vertical, F.Cu at (149.9, 110.3)
- added J15: 430450228, Connector_Molex:Molex_Micro-Fit_3.0_43045-0212_2x01_P3.00mm_Vertical, F.Cu at (225.8, 14.8)
- added J15: Conn_01x08, Connector_PinHeader_2.54mm:PinHeader_1x08_P2.54mm_Vertical, F.Cu at (137.2, 110.3)
- added J15: Extra I2C #3, Imported_Footprints:CONN_SD-43045-005_04_MOL, F.Cu at (273.5, 113.0)
- added J16: Extra I2C #6, Imported_Footprints:CONN_SD-43045-005_04_MOL, F.Cu at (273.5, 80.0)
- added J16: Conn_01x02_Pin, Connector_AMASS:AMASS_XT60PW-F_1x02_P7.20mm_Horizontal, F.Cu at (110.2, 84.9)
- added J17: Extra I2C #5, Imported_Footprints:CONN_SD-43045-005_04_MOL, F.Cu at (273.5, 91.0)
- added J18: Extra I2C #4, Imported_Footprints:CONN_SD-43045-005_04_MOL, F.Cu at (273.5, 102.0)
- added J18: Conn_01x04_Socket, Connector_Phoenix_MC:PhoenixContact_MCV_1,5_4-G-3.81_1x04_P3.81mm_Vertical, F.Cu at (142.1, 89.6)
- added J2: Conn_01x02_Pin, Connector_AMASS:AMASS_XT30PW-F_1x02_P2.50mm_Horizontal, F.Cu at (128.6, -4.66)
- added J2: Interconnect, Imported_Footprints:SULLINS_SBH11-PBPC-D05-ST-BK, F.Cu at (217.6, 112.2)
- added J21: 5V Line, Connector_PinHeader_2.54mm:PinHeader_1x10_P2.54mm_Vertical, F.Cu at (289.5, 74.3)
- added J21: Conn_01x02_Pin, Connector_AMASS:AMASS_XT60PW-F_1x02_P7.20mm_Horizontal, F.Cu at (102.8, 107.1)
- added J22: Conn_01x02_Pin, Connector_AMASS:AMASS_XT60PW-F_1x02_P7.20mm_Horizontal, F.Cu at (102.7, 90.3)
- added J22: Extra SPI #1, Imported_Footprints:CONN_SD-43045-005_06_MOL, F.Cu at (252.0, 144.5)
- added J3: External Battery, Connector_AMASS:AMASS_XT60PW-F_1x02_P7.20mm_Horizontal, F.Cu at (288.3, 143.7)
- added J3: SBH11-PBPC-D05-ST-BK, Imported_Footprints:SULLINS_SBH11-PBPC-D05-ST-BK, F.Cu at (189.1, -6.63)
- added J4: 1098169, Imported_Footprints:PHOENIX_1098169, F.Cu at (104.3, 65.3)
- added J4: Conn_01x24, Connector_PinHeader_2.54mm:PinHeader_1x24_P2.54mm_Vertical, F.Cu at (203.4, 97.9)
- added J5: External I2C, Connector_AMASS:AMASS_XT30PW-F_1x02_P2.50mm_Horizontal, F.Cu at (277.0, 143.8)
- added J5: 1098169, Imported_Footprints:PHOENIX_1098169, F.Cu at (136.3, 65.3)
- added J6: 1098169, Imported_Footprints:PHOENIX_1098169, F.Cu at (168.3, 65.3)
- added J6: Conn_01x24, Connector_PinHeader_2.54mm:PinHeader_1x24_P2.54mm_Vertical, F.Cu at (203.5, 75.4)
- added J7: Extra I2C #1, Imported_Footprints:CONN_SD-43045-005_04_MOL, F.Cu at (273.5, 135.0)
- added J7: 1098169, Imported_Footprints:PHOENIX_1098169, F.Cu at (200.3, 65.3)
- added J8: 0430450212, Connector_Molex:Molex_Micro-Fit_3.0_43045-0212_2x01_P3.00mm_Vertical, F.Cu at (155.8, 14.8)
- added J8: Extra I2C #2, Imported_Footprints:CONN_SD-43045-005_04_MOL, F.Cu at (273.5, 124.0)
- added J9: Lumen PWM, Imported_Footprints:CONN_SD-43045-005_02_MOL, F.Cu at (239.7, 127.6)
- added J9: 430450228, Connector_Molex:Molex_Micro-Fit_3.0_43045-0212_2x01_P3.00mm_Vertical, F.Cu at (165.8, 14.8)
- added J98: Conn_01x08, Connector_PinHeader_2.54mm:PinHeader_1x08_P2.54mm_Vertical, F.Cu at (168.3, 2.79)
- added J99: Conn_01x08, Connector_PinHeader_2.54mm:PinHeader_1x08_P2.54mm_Vertical, F.Cu at (168.3, -9.90)
- added Q7: L78M05ABDT-TR, robosub_footprints:TO-252-2_L6.5-W6.1-P4.58-LS10.0-TL, F.Cu at (155.2, 74.2)
- added Q7: L78M05ABDT-TR, robosub_footprints:TO-252-2_L6.5-W6.1-P4.58-LS10.0-TL, F.Cu at (295.5, 127.5)
- added Q7: L78M05ABDT-TR, robosub_footprints:TO-252-2_L6.5-W6.1-P4.58-LS10.0-TL, F.Cu at (128.9, 5.08)
- added R1: 10k, Resistor_SMD:R_0805_2012Metric_Pad1.20x1.40mm_HandSolder, F.Cu at (153.6, 8.85)
- added R1: 0R, Resistor_SMD:R_0805_2012Metric_Pad1.20x1.40mm_HandSolder, F.Cu at (288.5, 105.5)
- added R10: 10k, Resistor_SMD:R_0805_2012Metric_Pad1.20x1.40mm_HandSolder, F.Cu at (267.0, 89.5)
- added R11: 10k, Resistor_SMD:R_0805_2012Metric_Pad1.20x1.40mm_HandSolder, F.Cu at (267.0, 92.5)
- added R2: 10k, Resistor_SMD:R_0805_2012Metric_Pad1.20x1.40mm_HandSolder, F.Cu at (288.5, 102.5)
- added R2: 0R, Resistor_SMD:R_0805_2012Metric_Pad1.20x1.40mm_HandSolder, F.Cu at (159.7, -3.65)
- added R3: 2.2k Array, Imported_Footprints:2506_8x_Resistor_Array, F.Cu at (168.1, -3.65)
- added R3: 10k, Resistor_SMD:R_0805_2012Metric_Pad1.20x1.40mm_HandSolder, F.Cu at (284.5, 103.5)
- added R4: 3.3k Array, Imported_Footprints:2506_8x_Resistor_Array, F.Cu at (163.6, -3.65)
- added R4: 10k, Resistor_SMD:R_0805_2012Metric_Pad1.20x1.40mm_HandSolder, F.Cu at (285.5, 133.0)
- added R5: 0R, Resistor_SMD:R_0805_2012Metric_Pad1.20x1.40mm_HandSolder, F.Cu at (157.1, -3.65)
- added R5: 10k, Resistor_SMD:R_0805_2012Metric_Pad1.20x1.40mm_HandSolder, F.Cu at (288.4, 133.0)
- added R6: 0R, Resistor_SMD:R_0805_2012Metric_Pad1.20x1.40mm_HandSolder, F.Cu at (153.1, -3.56)
- added R6: 10k, Resistor_SMD:R_0805_2012Metric_Pad1.20x1.40mm_HandSolder, F.Cu at (267.0, 80.5)
- added R7: 10k, Resistor_SMD:R_0805_2012Metric_Pad1.20x1.40mm_HandSolder, F.Cu at (267.0, 83.5)
- added R7: 0R, Resistor_SMD:R_0805_2012Metric_Pad1.20x1.40mm_HandSolder, F.Cu at (143.9, -9.15)
- added R8: 10k, Resistor_SMD:R_0805_2012Metric_Pad1.20x1.40mm_HandSolder, F.Cu at (267.0, 86.5)
- added R8: 0R, Resistor_SMD:R_0805_2012Metric_Pad1.20x1.40mm_HandSolder, F.Cu at (143.8, -6.66)
- added U15: AMS1117-3.3, Package_TO_SOT_SMD:SOT-223-3_TabPin2, F.Cu at (294.5, 113.5)
- added U15: AMS1117-3.3, Package_TO_SOT_SMD:SOT-223-3_TabPin2, F.Cu at (158.5, 82.8)
- added U2: MCP9808_MSOP, Package_SO:MSOP-8_3x3mm_P0.65mm, F.Cu at (287.0, 123.0)
- added U4: BME280, Package_LGA:Bosch_LGA-8_2.5x2.5mm_P0.65mm_ClockwisePinNumbering, F.Cu at (294.5, 104.0)
- added U6: Teensy4.1, Imported_Footprints:Teensy41, F.Cu at (232.7, 86.6)
- C3, C5: value 10uF -> 1 µF; footprint Capacitor_SMD:C_0805_2012Metric_Pad1.18x1.45mm_HandSolder -> Capacitor_SMD:C_0805_2012Metric
- C4: value 10uF -> 10 µF; footprint Capacitor_SMD:C_0805_2012Metric_Pad1.18x1.45mm_HandSolder -> Capacitor_SMD:C_0805_2012Metric
- C6: value 1uF -> 10 µF; footprint Capacitor_SMD:C_0805_2012Metric_Pad1.18x1.45mm_HandSolder -> Capacitor_SMD:C_0805_2012Metric
- U1: value STPS5045SG-TR -> MCP9808_MSOP; footprint Imported_Footprints:D2PAK_STM -> Package_SO:MSOP-8_3x3mm_P0.65mm
- U3: value LTC1255CS8-PBF -> AMS1117-3.3; footprint Imported_Footprints:LTC1255 -> Package_TO_SOT_SMD:SOT-223-3_TabPin2
- moved J19 216.8 mm to (297.5, 74.2), turned to 0 degrees
- moved J20 209.3 mm to (293.5, 74.2), turned to 0 degrees
- moved D15 144.0 mm to (144.9, 72.0)
- moved R32 144.0 mm to (147.1, 110.5)
- moved R35 144.0 mm to (144.8, 118.6)
- moved C16 144.0 mm to (121.8, 122.7)
- moved C17 144.0 mm to (126.9, 123.3)
- moved C18 144.0 mm to (124.9, 123.2)
- moved C19 144.0 mm to (151.9, 80.1)
- moved C20 144.0 mm to (149.9, 80.1)
- moved D16 144.0 mm to (145.1, 76.1)
- moved R28 144.0 mm to (130.8, 123.2)
- moved R29 144.0 mm to (110.4, 115.0)
- moved R30 144.0 mm to (110.4, 113.0)
- moved R33 144.0 mm to (146.7, 114.5)
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Connections:
- C3 pad 1: +VregDiode -> +5V
- C3 pad 2: -BATT1 -> -BATT
- C4 pad 2: -BATT1 -> -BATT
- C5 pad 2: -BATT1 -> -BATT
- C6 pad 2: -BATT1 -> -BATT
- U1 pad 1: +BATT1 -> SDA
- U1 pad 2: +VregDiode -> SCL
- U1 pad 3: +BATT1 -> unconnected-(U1-Alert-Pad3)
- U3 pad 1: Net-(JP1-A) -> -BATT
- U3 pad 2: Batt1GatePreDiv -> +3.3V
- U3 pad 3: -BATT1 -> +5V
Routing:
- net -BATT: track 0.00 -> 384.2 mm, vias 0 -> 3
- net +BATT: track 22.7 -> 324.1 mm
- net GND: track 379.9 -> 110.1 mm, vias 0 -> 31
- net ISample5V: track 260.2 -> 0.00 mm
- net +3.3V: track 645.9 -> 438.9 mm, vias 20 -> 7
- net Batt2Gate: track 198.2 -> 0.00 mm, vias 6 -> 0
- net I2C1_SDA: track 451.1 -> 259.3 mm, vias 2 -> 3
- net +BATT2: track 171.3 -> 0.00 mm, vias 2 -> 0
- net I2C1_SCL: track 400.6 -> 233.5 mm
- net +BATT1: track 133.4 -> 0.00 mm, vias 2 -> 0
- net Batt1Enable: track 125.4 -> 0.00 mm
- net Batt1Gate: track 111.9 -> 0.00 mm
- net /ENABLE_BATT2: track 86.2 -> 0.00 mm, vias 2 -> 0
- net VIout8: track 0.00 -> 82.4 mm
- net SDA: track 0.00 -> 79.7 mm, vias 0 -> 2
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- removed copper zone on B.Cu, net +BATT
- removed copper zone on F.Cu, net +BATT1
- removed copper zone on F.Cu, net +BATT2
- removed copper zone on F.Cu, net +BATTHall
- removed copper zone on B.Cu, net -BATT1
- removed copper zone on F.Cu, net -BATT1
- removed copper zone on F.Cu, net Capacitors
Other:
- board size 261.2 x 259 mm -> 220.2 x 164.9 mm
- board text removed: "+Vo"
- board text removed: "180mm"
- board text removed: "ADC Splitter"
- board text removed: "BATT 1 ENABLE"
- board text removed: "BATT 1 GATE"
- board text removed: "BATT 2 GATE"
- board text removed: "BATT1"
- board text removed: "BATT1 FIX POINT"
- board text removed: "BATT2"
- board text removed: "BATT2 FIX POINT"
- board text removed: "BOTTOM SIDE OBSTRUCTED, LEFT RIGHT USED FOR SLIDING RAILS, POWER CONNECTORS AT THE TOP AND THE BUSSES ON THE SIDE"
- board text removed: "Batt1En"
- board text removed: "Batt1UVP"
- board text removed: "Batt2En"
- board text removed: "Batt2UVP"
- board text removed: "Enable"
- board text removed: "ExtKill"
- board text removed: "GATE DRIVER"
- board text removed: "GROUND"
- board text removed: "KillStatus"
- board text removed: "OCPLatch"
- board text removed: "Said Vassili on the first iteration of this..."
- board text removed: "Stanford Robosub Power Management"
- board text removed: "Switch"
- board text removed: "TVS DIODE"
- board text removed: "Vin"
- board text removed: "ballast resistance 7x14mm ~ 1mOhm"
- board text removed: "zener protection diodes (Vgs > 12V) the driver drives until the clamp is satisfied"
- board text removed: "{dblquote}Survival is the ability to swim in strange water{dblquote}"
