File: gen3/PCBs/Hydrophone/Hydrophone.kicad_sch (KiCad schematic)
At the start: 4 parts, among them J1 Conn_Coaxial, J2 Conn_Coaxial, J3 Conn_Coaxial, J4 Conn_Coaxial

Commit message: renamed Control_and_Relays sheet to Control
Other:
- sheet Control_and_Relays renamed Control
- sheet Control: file Control_and_Relays.kicad_sch -> Control.kicad_sch
Changed lines of the file:
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@@
 			(color 0 0 0 0)
 		)
-		(property "Sheetname" "Control_and_Relays"
+		(property "Sheetname" "Control"
 			(at 154.94 102.1584 0)
 			(show_name no)
@@
 			)
 		)
-		(property "Sheetfile" "Control_and_Relays.kicad_sch"
+		(property "Sheetfile" "Control.kicad_sch"
 			(at 154.94 145.3646 0)
 			(show_name no)
