File: gen3/PCBs/Hydrophone_Analog/Analog_Channel.kicad_sch (KiCad schematic)
At the start: 48 parts, among them K1 Relay_SPST-NO, K2 Relay_DPDT, K3 Relay_SPST-NO, K4 Relay_SPST-NO, K5 Relay_DPDT, U1 OPA1656ID, U2 OPA1656ID, U3 THS4551xRGT

Commit message: Finalized Hydrophone Analog and Power board schematics and power tree
Parts:
- C1, C10, C12, C13, C14, C15, C16, C2, C3, C4, C5, C6, C65, C7, C9: footprint (none) -> Capacitor_SMD:C_0805_2012Metric
- C11, C8: footprint (none) -> Capacitor_SMD:C_1206_3216Metric
- K1, K3, K4: footprint (none) -> Relay_THT:Relay_SPST_Schrack-RT1-FormA_RM5mm
- K2, K5: footprint (none) -> Relay_THT:Relay_DPDT_Schrack-RT2-FormC_RM5mm
- R1, R10, R11, R12, R13, R14, R15, R16, R17, R2, R3, R4, R5, R6, R7, R8, R9: footprint (none) -> Resistor_SMD:R_0805_2012Metric

Commit message: fixed labelling issues + power design choices, switched footprints to smaller relays
Parts:
- C11, C8: value 47uF -> 10uF
- C15, C4: value 82pF -> 820pF
- C16, C5: value 820pF -> 82pF
Changed lines of the file:
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@@
 	(wire
 		(pts
-			(xy 181.61 156.21) (xy 172.72 156.21)
+			(xy 181.61 157.48) (xy 172.72 157.48)
 		)
 		(stroke
@@
 	(wire
 		(pts
-			(xy 172.72 156.21) (xy 172.72 153.67)
+			(xy 172.72 157.48) (xy 172.72 153.67)
 		)
 		(stroke
@@
 	(wire
 		(pts
-			(xy 181.61 148.59) (xy 181.61 156.21)
+			(xy 181.61 148.59) (xy 181.61 157.48)
 		)
 		(stroke
@@
 	)
 	(label "-5VA"
-		(at 172.72 156.21 0)
+		(at 172.72 157.48 0)
 		(effects
 			(font
@@
 			)
 		)
-		(property "Value" "47uF"
+		(property "Value" "10uF"
 			(at 185.42 146.0499 0)
 			(show_name no)
@@
 			)
 		)
-		(property "Value" "82pF"
+		(property "Value" "820pF"
 			(at 86.36 101.5999 0)
 			(show_name no)
@@
 			)
 		)
-		(property "Value" "82pF"
+		(property "Value" "820pF"
 			(at 237.49 39.3699 0)
 			(show_name no)
@@
 			)
 		)
-		(property "Value" "820pF"
+		(property "Value" "82pF"
 			(at 250.19 39.3699 0)
 			(show_name no)
@@
 			)
 		)
-		(property "Value" "47uF"
+		(property "Value" "10uF"
 			(at 166.37 147.3199 0)
 			(show_name no)
@@
 			)
 		)
-		(property "Value" "820pF"
+		(property "Value" "82pF"
 			(at 99.06 101.5999 0)
 			(show_name no)
