File: gen3/PCBs/Hydrophone_Analog/Hydrophone_Analog.kicad_sch (KiCad schematic)
At the start: 4 parts, among them J1 Conn_Coaxial, J2 Conn_Coaxial, J3 Conn_Coaxial, J4 Conn_Coaxial

Commit message: Finalized Hydrophone Analog and Power board schematics and power tree
Parts:
- added J5: Conn_02x12_Odd_Even, Connector_PinHeader_2.54mm:PinHeader_2x12_P2.54mm_Vertical, symbol Connector_Generic:Conn_02x12_Odd_Even
- J1, J2, J3, J4: footprint (none) -> Connector_PinHeader_2.54mm:PinHeader_1x02_P2.54mm_Vertical
Connections:
- net CH0_AINN: now also J5.3 (Pin_3)
- net CH0_AINP: now also J5.1 (Pin_1)
- net CH1_AINN: now also J5.7 (Pin_7)
- net CH1_AINP: now also J5.5 (Pin_5)
- net CH2_AINN: now also J5.11 (Pin_11)
- net CH2_AINP: now also J5.9 (Pin_9)
- net CH3_AINN: now also J5.15 (Pin_15)
- net CH3_AINP: now also J5.13 (Pin_13)
- net VOCM: now also J5.17 (Pin_17)
- net AGND renamed GND
- net GND: now also J5.10 (Pin_10), J5.12 (Pin_12), J5.14 (Pin_14), J5.16 (Pin_16), J5.18 (Pin_18), J5.2 (Pin_2), J5.22 (Pin_22), J5.4 (Pin_4), J5.6 (Pin_6), J5.8 (Pin_8)
- new net +5V: J5.19 (Pin_19)
- new net +VCOIL: J5.20 (Pin_20)
- new net 12C1_SCL: J5.21 (Pin_21)
- new net 12C1_SDA: J5.23 (Pin_23)
- new net CTRL_RESET_N: J5.24 (Pin_24)
Other:
- removed sheet ADC_and_Digital
- sheet Control ports: added CH0_FILT_AUDIO, CH0_GAIN_G11, CH0_GAIN_G2, CH0_RX_EN, CH1_FILT_AUDIO, CH1_GAIN_G11, CH1_GAIN_G2, CH1_RX_EN, CH2_FILT_AUDIO, CH2_GAIN_G11, CH2_GAIN_G2, CH2_RX_EN, CH3_FILT_AUDIO, CH3_GAIN_G11, CH3_GAIN_G2, CH3_RX_EN; removed none

Commit message: fixed labelling issues + power design choices, switched footprints to smaller relays
Connections:
- net 12C1_SCL is gone; now on net I2C1_SCL: J5.21 (Pin_21)
- net 12C1_SDA is gone; now on net I2C1_SDA: J5.23 (Pin_23)
Other:
- sheet Control ports: added CTRL_RESET_N, I2C1_SCL, I2C1_SDA; removed none
Changed lines of the file:
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@@
 	(wire
 		(pts
-			(xy 210.82 111.76) (xy 228.6 111.76)
+			(xy 38.1 52.07) (xy 43.18 52.07)
 		)
 		(stroke
@@
 	(wire
 		(pts
-			(xy 38.1 52.07) (xy 43.18 52.07)
+			(xy 43.18 165.1) (xy 44.45 165.1)
 		)
 		(stroke
@@
 	(wire
 		(pts
-			(xy 43.18 165.1) (xy 44.45 165.1)
+			(xy 151.13 115.57) (xy 154.94 115.57)
 		)
 		(stroke
@@
 	(wire
 		(pts
-			(xy 151.13 115.57) (xy 154.94 115.57)
+			(xy 43.18 55.88) (xy 38.1 55.88)
 		)
 		(stroke
@@
 	(wire
 		(pts
-			(xy 43.18 55.88) (xy 38.1 55.88)
+			(xy 151.13 133.35) (xy 154.94 133.35)
 		)
 		(stroke
@@
 	(wire
 		(pts
-			(xy 151.13 133.35) (xy 154.94 133.35)
+			(xy 212.09 111.76) (xy 228.6 111.76)
 		)
 		(stroke
@@
 	(wire
 		(pts
-			(xy 210.82 109.22) (xy 228.6 109.22)
-		)
-		(stroke
-			(width 0)
-			(type default)
-		)
-	)
-	(wire
-		(pts
 			(xy 347.98 156.21) (xy 353.06 156.21)
 		)
@@
 	(wire
 		(pts
+			(xy 212.09 105.41) (xy 228.6 105.41)
+		)
+		(stroke
+			(width 0)
+			(type default)
+		)
+	)
+	(wire
+		(pts
 			(xy 347.98 151.13) (xy 353.06 151.13)
 		)
@@
 	(wire
 		(pts
-			(xy 210.82 105.41) (xy 228.6 105.41)
-		)
-		(stroke
-			(width 0)
-			(type default)
-		)
-	)
-	(wire
-		(pts
 			(xy 43.18 218.44) (xy 44.45 218.44)
 		)
@@
 	(wire
 		(pts
+			(xy 212.09 109.22) (xy 228.6 109.22)
+		)
+		(stroke
+			(width 0)
+			(type default)
+		)
+	)
+	(wire
+		(pts
 			(xy 347.98 153.67) (xy 353.06 153.67)
 		)
@@
 		)
 	)
-	(label "CH0_GAIN_G2"
+	(label "CH1_GAIN_G2"
 		(at 38.1 104.14 180)
 		(effects
@@
 		)
 	)
-	(label "12C1_SDA"
+	(label "I2C1_SDA"
 		(at 347.98 156.21 180)
 		(effects
@@
 		)
 	)
-	(label "CH0_FILT_AUDIO"
+	(label "CH1_FILT_AUDIO"
 		(at 39.37 99.06 180)
 		(effects
@@
 		)
 	)
-	(label "12C1_SCL"
+	(label "I2C1_SCL"
 		(at 347.98 153.67 180)
 		(effects
@@
 		)
 	)
-	(label "I2C1_SDA"
-		(at 210.82 109.22 0)
-		(effects
-			(font
-				(size 1.27 1.27)
-			)
-			(justify left bottom)
-		)
-	)
 	(label "CH1_GAIN_G2"
 		(at 151.13 120.65 180)
@@
 		)
 	)
-	(label "CH0_RX_EN"
+	(label "CH1_RX_EN"
 		(at 39.37 115.57 180)
 		(effects
@@
 		)
 	)
-	(label "CH0_GAIN_G11"
+	(label "CH1_GAIN_G11"
 		(at 39.37 107.95 180)
 		(effects
@@
 		)
 	)
-	(hierarchical_label "I2C1_SCL"
-		(shape input)
-		(at 210.82 105.41 0)
-		(effects
-			(font
-				(size 1.27 1.27)
-			)
-			(justify left)
-		)
-	)
-	(hierarchical_label "CTRL_RESET_N"
-		(shape input)
-		(at 210.82 111.76 0)
-		(effects
-			(font
-				(size 1.27 1.27)
-			)
-			(justify left)
-		)
-	)
 	(symbol
 		(lib_id "power:GND")
@@
 			)
 		)
-		(pin "CH0_GAIN_G11" input
+		(pin "CH0_GAIN_G11" output
 			(at 154.94 107.95 180)
 			(effects
@@
 			)
 		)
+		(pin "CTRL_RESET_N" input
+			(at 212.09 111.76 0)
+			(effects
+				(font
+					(size 1.27 1.27)
+				)
+				(justify right)
+			)
+		)
+		(pin "I2C1_SCL" input
+			(at 212.09 105.41 0)
+			(effects
+				(font
+					(size 1.27 1.27)
+				)
+				(justify right)
+			)
+		)
+		(pin "I2C1_SDA" input
+			(at 212.09 109.22 0)
+			(effects
+				(font
+					(size 1.27 1.27)
+				)
+				(justify right)
+			)
+		)
