File: gen3/PCBs/Hydrophone_Analog/Power_Supply.kicad_sch (KiCad schematic)
At the start: 0 parts

Commit message: Finalized Hydrophone Analog and Power board schematics and power tree
Parts:
- added C69, C71, C72, C73, C74, C76, C77, C79: 10uF, Capacitor_SMD:C_1206_3216Metric, symbol Device:C
- added C70: 22uF, Capacitor_SMD:C_1206_3216Metric, symbol Device:C
- added C75, C78: 100nF, Capacitor_SMD:C_0805_2012Metric, symbol Device:C
- added J6: Conn_01x02, TerminalBlock_Phoenix:TerminalBlock_Phoenix_MKDS-1,5-2-5.08_1x02_P5.08mm_Horizontal, symbol Connector_Generic:Conn_01x02
- added U13: ICL7660, Package_SO:SOIC-8_3.9x4.9mm_P1.27mm, symbol Regulator_SwitchedCapacitor:ICL7660
- added U7: R-78E5.0-1.0, Converter_DCDC:Converter_DCDC_RECOM_R-78E-0.5_THT, symbol Converter_DCDC:R-78E5.0-1.0
- added U8: AMS1117-3.3, Package_TO_SOT_SMD:SOT-223-3_TabPin2, symbol Regulator_Linear:AMS1117-3.3
- added U9: L7805, Package_TO_SOT_SMD:TO-252-2, symbol Regulator_Linear:L7805
Connections:
- new net: C79.1, U13.2 (CAP+)
- new net: C79.2, U13.4 (CAP-)
- new net +3.3V: C72.1, U8.2 (VO)
- new net +5V: C74.1, C75.1, U9.3 (OUT)
- new net +VBAT: C69.1, J6.1 (Pin_1), U7.1 (IN)
- new net +VCOIL: C70.1, C71.1, C73.1, C76.1, U13.8 (V+), U7.3 (OUT), U8.3 (VI), U9.1 (IN)
- new net -5V: C77.1, C78.1, U13.5 (VOUT)
- new net GND: C69.2, C70.2, C71.2, C72.2, C73.2, C74.2, C75.2, C76.2, C77.2, C78.2, J6.2 (Pin_2), U13.3 (GND), U7.2 (GND), U8.1 (GND), U9.2 (GND)

Commit message: fixed labelling issues + power design choices, switched footprints to smaller relays
Parts:
- removed C79: 10uF, Capacitor_SMD:C_1206_3216Metric, symbol Device:C
- removed U13: ICL7660, Package_SO:SOIC-8_3.9x4.9mm_P1.27mm, symbol Regulator_SwitchedCapacitor:ICL7660
- added U14: R-78E5.0-0.5, Converter_DCDC:Converter_DCDC_RECOM_R-78E-0.5_THT, symbol Converter_DCDC:R-78E5.0-0.5
Connections:
- net +VBAT: now also C73.1, C76.1, U9.1 (IN), U14.1 (IN)
- net +VCOIL: no longer C73.1, C76.1, U9.1 (IN)
- net -5V: now also U14.2 (GND)
- net GND: now also U14.3 (OUT)
